File: Hardware/SparkFun_ProMicro_RP2350.sch (EAGLE design)
At the start: 61 parts, among them J2 QWIIC_RIGHT_ANGLE, J5 USB Female Type C Connector, U1 RT9080-33GJ5, U2 RP2350A, U3 WS2812_2020, U4 W25QXX128MBIT, Y1 12MHz

Commit message: Design review updates
Change all text and labels in schematic to vector font
Fix overlapping text with Qwiic connector in schematic
Add part number to flash memory section title
Fix acid trap on RAW pad
Add more GND vias
Other:
- note added: "16MB Flash - W25Q128"
- note removed: "16MB Flash"
