File: Production/SparkFun_ProMicro_RP2350-Panel.brd (EAGLE design)
At the start: 92.7 x 87.1 mm, 702 parts, among them J1 QWIIC_RIGHT_ANGLE, J12 USB Female Type C Connector, J13 QWIIC_RIGHT_ANGLE, J16 USB Female Type C Connector, J17 QWIIC_RIGHT_ANGLE, J2 QWIIC_RIGHT_ANGLE, J20 USB Female Type C Connector, J21 QWIIC_RIGHT_ANGLE, J24 USB Female Type C Connector, J5 USB Female Type C Connector, J8 USB Female Type C Connector, J9 QWIIC_RIGHT_ANGLE, U1 RT9080-33GJ5, U10 W25QXX128MBIT, U11 WS2812_2020, U12 RP2350A, U13 RT9080-33GJ5, U14 W25QXX128MBIT, U15 WS2812_2020, U16 RP2350A, U17 RT9080-33GJ5, U18 W25QXX128MBIT, U19 WS2812_2020, U2 RP2350A, U20 RP2350A, U21 RT9080-33GJ5, U22 W25QXX128MBIT, U23 WS2812_2020, U24 RP2350A, U3 WS2812_2020, U4 W25QXX128MBIT, U5 RT9080-33GJ5, U6 W25QXX128MBIT, U7 WS2812_2020, U8 RP2350A, U9 RT9080-33GJ5, Y1 12MHz, Y2 12MHz, Y3 12MHz, Y4 12MHz, Y5 12MHz, Y6 12MHz

Commit message: Add v10 production files
Parts:
- added C115, C116, C127, C128, C134, C135, C146, C147, C153, C154, C165, C166, C172, C173, C184, C185, C191, C192, C203, C204, C210, C211, C222, C223, C229, C230, C241, C242, C248, C249, C260, C261, C267, C268, C279, C280, C286, C287, C298, C299, C305, C306, C317, C318, C324, C325, C336, C337, C343, C344, C355, C356, C362, C363, C374, C375, C381, C382, C393, C394, C400, C401, C412, C413, C419, C420, C431, C432, C438, C439, C450, C451: 10uF, SparkFun-Capacitors:0402-TIGHT
- added C117, C118, C136, C137, C155, C156, C174, C175, C193, C194, C212, C213, C231, C232, C250, C251, C269, C270, C288, C289, C307, C308, C326, C327, C345, C346, C364, C365, C383, C384, C402, C403, C421, C422, C440, C441: 15pF, SparkFun-Capacitors:0402-TIGHT
- added C119, C120, C121, C122, C123, C124, C125, C126, C130, C132, C133, C138, C139, C140, C141, C142, C143, C144, C145, C149, C151, C152, C157, C158, C159, C160, C161, C162, C163, C164, C168, C170, C171, C176, C177, C178, C179, C180, C181, C182, C183, C187, C189, C190, C195, C196, C197, C198, C199, C200, C201, C202, C206, C208, C209, C214, C215, C216, C217, C218, C219, C220, C221, C225, C227, C228, C233, C234, C235, C236, C237, C238, C239, C240, C244, C246, C247, C252, C253, C254, C255, C256, C257, C258, C259, C263, C265, C266, C271, C272, C273, C274, C275, C276, C277, C278, C282, C284, C285, C290, C291, C292, C293, C294, C295, C296, C297, C301, C303, C304, C309, C310, C311, C312, C313, C314, C315, C316, C320, C322, C323, C328, C329, C330, C331, C332, C333, C334, C335, C339, C341, C342, C347, C348, C349, C350, C351, C352, C353, C354, C358, C360, C361, C366, C367, C368, C369, C370, C371, C372, C373, C377, C379, C380, C385, C386, C387, C388, C389, C390, C391, C392, C396, C398, C399, C404, C405, C406, C407, C408, C409, C410, C411, C415, C417, C418, C423, C424, C425, C426, C427, C428, C429, C430, C434, C436, C437, C442, C443, C444, C445, C446, C447, C448, C449, C453, C455, C456: 0.1uF, SparkFun-Capacitors:0402-TIGHT
- added C129, C131, C148, C150, C167, C169, C186, C188, C205, C207, C224, C226, C243, C245, C262, C264, C281, C283, C300, C302, C319, C321, C338, C340, C357, C359, C376, C378, C395, C397, C414, C416, C433, C435, C452, C454: 2.2uF, SparkFun-Capacitors:0402-TIGHT
- added D10, D11, D12, D13, D14, D15, D16, D17, D18, D19, D20, D21, D22, D23, D24, D7, D8, D9: 3A/10V/280mV, SparkFun-DiscreteSemi:SOD-323
- added F10, F11, F12, F13, F14, F15, F16, F17, F18, F19, F20, F21, F22, F23, F24, F7, F8, F9: 6V 0.5A, SparkFun-Fuses:0805
- added J25, J29, J33, J37, J41, J45, J49, J53, J57, J61, J65, J69, J73, J77, J81, J85, J89, J93: QWIIC_RIGHT_ANGLE, SparkFun-Connectors:JST04_1MM_RA
- added J26, J27, J30, J31, J34, J35, J38, J39, J42, J43, J46, J47, J50, J51, J54, J55, J58, J59, J62, J63, J66, J67, J70, J71, J74, J75, J78, J79, J82, J83, J86, J87, J90, J91, J94, J95: (no value), SparkFun-Connectors:1X12_CASTELLATED
- added J28, J32, J36, J40, J44, J48, J52, J56, J60, J64, J68, J72, J76, J80, J84, J88, J92, J96: USB Female Type C Connector, SparkFun-Connectors:USB-C-16P_4LAYER-PADS
- added JP19, JP20, JP22, JP23, JP25, JP26, JP28, JP29, JP31, JP32, JP34, JP35, JP37, JP38, JP40, JP41, JP43, JP44, JP46, JP47, JP49, JP50, JP52, JP53, JP55, JP56, JP58, JP59, JP61, JP62, JP64, JP65, JP67, JP68, JP70, JP71: FIDUCIAL1X2, SparkFun-Aesthetics:FIDUCIAL-1X2
- added JP21, JP24, JP27, JP30, JP33, JP36, JP39, JP42, JP45, JP48, JP51, JP54, JP57, JP60, JP63, JP66, JP69, JP72: USB_SOLDER_PADS, SparkFun-Connectors:USB-SOLDER-PADS
- added L10, L11, L12, L13, L14, L15, L16, L17, L18, L19, L20, L21, L22, L23, L24, L7, L8, L9: 4.7μH, SparkFun-Coils:1008(2520)
- added LED10, LED11, LED12, LED13, LED14, LED15, LED16, LED17, LED18, LED19, LED20, LED21, LED22, LED23, LED24, LED7, LED8, LED9: Red, SparkFun-LED:LED-0603
- added LOGO19, LOGO22, LOGO25, LOGO28, LOGO31, LOGO34, LOGO37, LOGO40, LOGO43, LOGO46, LOGO49, LOGO52, LOGO55, LOGO58, LOGO61, LOGO64, LOGO67, LOGO70: SFE_LOGO_NAME_FLAME.1_INCH, SparkFun-Aesthetics:SFE_LOGO_NAME_FLAME_.1
- added LOGO20, LOGO23, LOGO26, LOGO29, LOGO32, LOGO35, LOGO38, LOGO41, LOGO44, LOGO47, LOGO50, LOGO53, LOGO56, LOGO59, LOGO62, LOGO65, LOGO68, LOGO71: QWIIC_LOGO_6MM, SparkFun-Aesthetics:QWIIC_6MM
- added LOGO21, LOGO24, LOGO27, LOGO30, LOGO33, LOGO36, LOGO39, LOGO42, LOGO45, LOGO48, LOGO51, LOGO54, LOGO57, LOGO60, LOGO63, LOGO66, LOGO69, LOGO72: SFE_LOGO_FLAME.1_INCH, SparkFun-Aesthetics:SFE_LOGO_FLAME_.1
- added PWR10, PWR11, PWR12, PWR13, PWR14, PWR15, PWR16, PWR17, PWR18, PWR19, PWR20, PWR21, PWR22, PWR23, PWR6, PWR7, PWR8, PWR9, SHLD10, SHLD11, SHLD12, SHLD13, SHLD14, SHLD15, SHLD16, SHLD17, SHLD18, SHLD19, SHLD20, SHLD21, SHLD22, SHLD23, SHLD6, SHLD7, SHLD8, SHLD9: JUMPER-SMT_2_NC_TRACE_SILK, SparkFun-Jumpers:SMT-JUMPER_2_NC_TRACE_SILK
- added R100, R111, R112, R123, R124, R135, R136, R147, R148, R159, R160, R171, R172, R183, R184, R195, R196, R207, R208, R219, R220, R231, R232, R243, R244, R255, R256, R267, R268, R279, R280, R75, R76, R87, R88, R99: 5.1k, SparkFun-Resistors:0402-TIGHT
- added R101, R102, R113, R114, R125, R126, R137, R138, R149, R150, R161, R162, R173, R174, R185, R186, R197, R198, R209, R210, R221, R222, R233, R234, R245, R246, R257, R258, R269, R270, R281, R282, R77, R78, R89, R90: 2.2k, SparkFun-Resistors:0402-TIGHT
- added R103, R107, R115, R119, R127, R131, R139, R143, R151, R155, R163, R167, R175, R179, R187, R191, R199, R203, R211, R215, R223, R227, R235, R239, R247, R251, R259, R263, R271, R275, R283, R287, R79, R83, R91, R95: 1k, SparkFun-Resistors:0402-TIGHT
- added R104, R105, R116, R117, R128, R129, R140, R141, R152, R153, R164, R165, R176, R177, R188, R189, R200, R201, R212, R213, R224, R225, R236, R237, R248, R249, R260, R261, R272, R273, R284, R285, R80, R81, R92, R93: 27, SparkFun-Resistors:0402-TIGHT
- added R106, R118, R130, R142, R154, R166, R178, R190, R202, R214, R226, R238, R250, R262, R274, R286, R82, R94: 10Ω, SparkFun-Resistors:0402-TIGHT
- added R108, R110, R120, R122, R132, R134, R144, R146, R156, R158, R168, R170, R180, R182, R192, R194, R204, R206, R216, R218, R228, R230, R240, R242, R252, R254, R264, R266, R276, R278, R288, R74, R84, R86, R96, R98: 10k, SparkFun-Resistors:0402-TIGHT
- added R109, R121, R133, R145, R157, R169, R181, R193, R205, R217, R229, R241, R253, R265, R277, R73, R85, R97: 4.7k, SparkFun-Resistors:0402-TIGHT
- added S13, S15, S17, S19, S21, S23, S25, S27, S29, S31, S33, S35, S37, S39, S41, S43, S45, S47: Reset, SparkFun-Switches:TACTILE_SWITCH_SMD_4.6X2.8MM
- added S14, S16, S18, S20, S22, S24, S26, S28, S30, S32, S34, S36, S38, S40, S42, S44, S46, S48: Boot, SparkFun-Switches:TACTILE_SWITCH_SMD_4.6X2.8MM
- added TP25, TP26, TP27, TP28, TP29, TP30, TP31, TP32, TP33, TP34, TP35, TP36, TP37, TP38, TP39, TP40, TP41, TP42, TP43, TP44, TP45, TP46, TP47, TP48, TP49, TP50, TP51, TP52, TP53, TP54, TP55, TP56, TP57, TP58, TP59, TP60, TP61, TP62, TP63, TP64, TP65, TP66, TP67, TP68, TP69, TP70, TP71, TP72, TP73, TP74, TP75, TP76, TP77, TP78, TP79, TP80, TP81, TP82, TP83, TP84, TP85, TP86, TP87, TP88, TP89, TP90, TP91, TP92, TP93, TP94, TP95, TP96: TEST-POINT3X5, SparkFun-Connectors:PAD.03X.05
- added U$1000, U$1058, U$1116, U$1174, U$1232, U$1290, U$1348, U$362, U$420, U$478, U$536, U$594, U$652, U$710, U$768, U$826, U$884, U$942: (no value), output:#RST#1
- added U$1001, U$1059, U$1117, U$1175, U$1233, U$1291, U$1349, U$363, U$421, U$479, U$537, U$595, U$653, U$711, U$769, U$827, U$885, U$943: (no value), output:3V30
- added U$1002, U$1060, U$1118, U$1176, U$1234, U$1292, U$1350, U$364, U$422, U$480, U$538, U$596, U$654, U$712, U$770, U$828, U$886, U$944: (no value), output:PWR0
- added U$1003, U$1018, U$1031, U$1061, U$1076, U$1089, U$1119, U$1134, U$1147, U$1177, U$1192, U$1205, U$1235, U$1250, U$1263, U$1293, U$1308, U$1321, U$1351, U$1366, U$1379, U$365, U$380, U$393, U$423, U$438, U$451, U$481, U$496, U$509, U$539, U$554, U$567, U$597, U$612, U$625, U$655, U$670, U$683, U$713, U$728, U$741, U$771, U$786, U$799, U$829, U$844, U$857, U$887, U$902, U$915, U$945, U$960, U$973: (no value), output:GND2
- added U$1004, U$1017, U$1062, U$1075, U$1120, U$1133, U$1178, U$1191, U$1236, U$1249, U$1294, U$1307, U$1352, U$1365, U$366, U$379, U$424, U$437, U$482, U$495, U$540, U$553, U$598, U$611, U$656, U$669, U$714, U$727, U$772, U$785, U$830, U$843, U$888, U$901, U$946, U$959: (no value), output:RX1
- added U$1005, U$1016, U$1063, U$1074, U$1121, U$1132, U$1179, U$1190, U$1237, U$1248, U$1295, U$1306, U$1353, U$1364, U$367, U$378, U$425, U$436, U$483, U$494, U$541, U$552, U$599, U$610, U$657, U$668, U$715, U$726, U$773, U$784, U$831, U$842, U$889, U$900, U$947, U$958: (no value), output:TX0
- added U$1006, U$1064, U$1122, U$1180, U$1238, U$1296, U$1354, U$368, U$426, U$484, U$542, U$600, U$658, U$716, U$774, U$832, U$890, U$948: (no value), output:GND_0
- added U$1007, U$1065, U$1123, U$1181, U$1239, U$1297, U$1355, U$369, U$427, U$485, U$543, U$601, U$659, U$717, U$775, U$833, U$891, U$949: (no value), output:70
- added U$1008, U$1066, U$1124, U$1182, U$1240, U$1298, U$1356, U$370, U$428, U$486, U$544, U$602, U$660, U$718, U$776, U$834, U$892, U$950: (no value), output:81
- added U$1009, U$1067, U$1125, U$1183, U$1241, U$1299, U$1357, U$371, U$429, U$487, U$545, U$603, U$661, U$719, U$777, U$835, U$893, U$951: (no value), output:92
- added U$1010, U$1050, U$1068, U$1108, U$1126, U$1166, U$1184, U$1224, U$1242, U$1282, U$1300, U$1340, U$1358, U$354, U$372, U$412, U$430, U$470, U$488, U$528, U$546, U$586, U$604, U$644, U$662, U$702, U$720, U$760, U$778, U$818, U$836, U$876, U$894, U$934, U$952, U$992: (no value), output:CI4
- added U$1011, U$1052, U$1069, U$1110, U$1127, U$1168, U$1185, U$1226, U$1243, U$1284, U$1301, U$1342, U$1359, U$356, U$373, U$414, U$431, U$472, U$489, U$530, U$547, U$588, U$605, U$646, U$663, U$704, U$721, U$762, U$779, U$820, U$837, U$878, U$895, U$936, U$953, U$994: (no value), output:SCK3
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Connections:
- new net !RESET!10: J43.3, J43.3B, R122.1, S21.3, S21.4, U44.26
- new net !RESET!11: J47.3, J47.3B, R134.1, S23.3, S23.4, U48.26
- new net !RESET!12: J51.3, J51.3B, R146.1, S25.3, S25.4, U52.26
- new net !RESET!13: J55.3, J55.3B, R158.1, S27.3, S27.4, U56.26
- new net !RESET!14: J59.3, J59.3B, R170.1, S29.3, S29.4, U60.26
- new net !RESET!15: J63.3, J63.3B, R182.1, S31.3, S31.4, U64.26
- new net !RESET!16: J67.3, J67.3B, R194.1, S33.3, S33.4, U68.26
- new net !RESET!17: J71.3, J71.3B, R206.1, S35.3, S35.4, U72.26
- new net !RESET!18: J75.3, J75.3B, R218.1, S37.3, S37.4, U76.26
- new net !RESET!19: J79.3, J79.3B, R230.1, S39.3, S39.4, U80.26
- new net !RESET!20: J83.3, J83.3B, R242.1, S41.3, S41.4, U84.26
- new net !RESET!21: J87.3, J87.3B, R254.1, S43.3, S43.4, U88.26
- new net !RESET!22: J91.3, J91.3B, R266.1, S45.3, S45.4, U92.26
- new net !RESET!23: J95.3, J95.3B, R278.1, S47.3, S47.4, U96.26
- new net !RESET!6: J27.3, J27.3B, R74.1, S13.3, S13.4, U28.26
- new net !RESET!7: J31.3, J31.3B, R86.1, S15.3, S15.4, U32.26
- new net !RESET!8: J35.3, J35.3B, R98.1, S17.3, S17.4, U36.26
- new net !RESET!9: J39.3, J39.3B, R110.1, S19.3, S19.4, U40.26
- new net 0/TX10: J42.12, J42.12B, U44.2
- new net 0/TX11: J46.12, J46.12B, U48.2
- new net 0/TX12: J50.12, J50.12B, U52.2
- new net 0/TX13: J54.12, J54.12B, U56.2
- new net 0/TX14: J58.12, J58.12B, U60.2
- new net 0/TX15: J62.12, J62.12B, U64.2
- new net 0/TX16: J66.12, J66.12B, U68.2
- new net 0/TX17: J70.12, J70.12B, U72.2
- new net 0/TX18: J74.12, J74.12B, U76.2
- new net 0/TX19: J78.12, J78.12B, U80.2
- new net 0/TX20: J82.12, J82.12B, U84.2
- new net 0/TX21: J86.12, J86.12B, U88.2
- new net 0/TX22: J90.12, J90.12B, U92.2
- new net 0/TX23: J94.12, J94.12B, U96.2
- new net 0/TX6: J26.12, J26.12B, U28.2
- new net 0/TX7: J30.12, J30.12B, U32.2
- new net 0/TX8: J34.12, J34.12B, U36.2
- new net 0/TX9: J38.12, J38.12B, U40.2
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Routing:
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- added copper zone on layer 1, net 1.1V10
- added copper zone on layer 1, net 1.1V11
- added copper zone on layer 1, net 1.1V12
- added copper zone on layer 1, net 1.1V13
- added copper zone on layer 1, net 1.1V14
- added copper zone on layer 1, net 1.1V15
- added copper zone on layer 1, net 1.1V16
- added copper zone on layer 1, net 1.1V17
- added copper zone on layer 1, net 1.1V18
- added copper zone on layer 1, net 1.1V19
- added copper zone on layer 1, net 1.1V20
- added copper zone on layer 1, net 1.1V21
- added copper zone on layer 1, net 1.1V22
- added copper zone on layer 1, net 1.1V23
- added copper zone on layer 1, net 1.1V6
- added copper zone on layer 1, net 1.1V7
- added copper zone on layer 1, net 1.1V8
- added copper zone on layer 1, net 1.1V9
- added copper zone on layer 1, net 3.3V10
- added copper zone on layer 15, net 3.3V10
- added copper zone on layer 1, net 3.3V11
- added copper zone on layer 15, net 3.3V11
- added copper zone on layer 1, net 3.3V12
- added copper zone on layer 15, net 3.3V12
- added copper zone on layer 1, net 3.3V13
- added copper zone on layer 15, net 3.3V13
- added copper zone on layer 1, net 3.3V14
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Other:
- board size 92.7 x 87.1 mm -> 207 x 125.5 mm
- board text added: "v10"
- board text removed: "v01"

Commit message: Add v09 panel files
Parts:
- removed C121, C122, C123, C124, C125, C126, C130, C132, C133, C138, C139, C140, C141, C142, C143, C144, C145, C149, C151, C152, C157, C158, C159, C160, C161, C162, C163, C164, C168, C170, C171, C176, C177, C178, C179, C180, C181, C182, C183, C187, C189, C190, C195, C196, C197, C198, C199, C200, C201, C202, C206, C208, C209, C214, C215, C216, C217, C218, C219, C220, C221, C225, C227, C228, C233, C234, C235, C236, C237, C238, C239, C240, C244, C246, C247, C252, C253, C254, C255, C256, C257, C258, C259, C263, C265, C266, C271, C272, C273, C274, C275, C276, C277, C278, C282, C284, C285, C290, C291, C292, C293, C294, C295, C296, C297, C301, C303, C304, C309, C310, C311, C312, C313, C314, C315, C316, C320, C322, C323, C328, C329, C330, C331, C332, C333, C334, C335, C339, C341, C342, C347, C348, C349, C350, C351, C352, C353, C354, C358, C360, C361, C366, C367, C368, C369, C370, C371, C372, C373, C377, C379, C380, C385, C386, C387, C388, C389, C390, C391, C392, C396, C398, C399, C404, C405, C406, C407, C408, C409, C410, C411, C415, C417, C418, C423, C424, C425, C426, C427, C428, C429, C430, C434, C436, C437, C442, C443, C444, C445, C446, C447, C448, C449, C453, C455, C456: 0.1uF, SparkFun-Capacitors:0402-TIGHT
- removed C127, C128, C134, C135, C146, C147, C153, C154, C165, C166, C172, C173, C184, C185, C191, C192, C203, C204, C210, C211, C222, C223, C229, C230, C241, C242, C248, C249, C260, C261, C267, C268, C279, C280, C286, C287, C298, C299, C305, C306, C317, C318, C324, C325, C336, C337, C343, C344, C355, C356, C362, C363, C374, C375, C381, C382, C393, C394, C400, C401, C412, C413, C419, C420, C431, C432, C438, C439, C450, C451: 10uF, SparkFun-Capacitors:0402-TIGHT
- removed C129, C131, C148, C150, C167, C169, C186, C188, C205, C207, C224, C226, C243, C245, C262, C264, C281, C283, C300, C302, C319, C321, C338, C340, C357, C359, C376, C378, C395, C397, C414, C416, C433, C435, C452, C454: 2.2uF, SparkFun-Capacitors:0402-TIGHT
- removed C136, C137, C155, C156, C174, C175, C193, C194, C212, C213, C231, C232, C250, C251, C269, C270, C288, C289, C307, C308, C326, C327, C345, C346, C364, C365, C383, C384, C402, C403, C421, C422, C440, C441: 15pF, SparkFun-Capacitors:0402-TIGHT
- removed D10, D11, D12, D13, D14, D15, D16, D17, D18, D19, D20, D21, D22, D23, D24, D7, D8, D9: 3A/10V/280mV, SparkFun-DiscreteSemi:SOD-323
- removed F10, F11, F12, F13, F14, F15, F16, F17, F18, F19, F20, F21, F22, F23, F24, F7, F8, F9: 6V 0.5A, SparkFun-Fuses:0805
- removed J25, J29, J33, J37, J41, J45, J49, J53, J57, J61, J65, J69, J73, J77, J81, J85, J89, J93: QWIIC_RIGHT_ANGLE, SparkFun-Connectors:JST04_1MM_RA
- removed J26, J27, J30, J31, J34, J35, J38, J39, J42, J43, J46, J47, J50, J51, J54, J55, J58, J59, J62, J63, J66, J67, J70, J71, J74, J75, J78, J79, J82, J83, J86, J87, J90, J91, J94, J95: (no value), SparkFun-Connectors:1X12_CASTELLATED
- removed J28, J32, J36, J40, J44, J48, J52, J56, J60, J64, J68, J72, J76, J80, J84, J88, J92, J96: USB Female Type C Connector, SparkFun-Connectors:USB-C-16P_4LAYER-PADS
- removed JP31, JP32, JP34, JP35, JP37, JP38, JP40, JP41, JP43, JP44, JP46, JP47, JP49, JP50, JP52, JP53, JP55, JP56, JP58, JP59, JP61, JP62, JP64, JP65, JP67, JP68, JP70, JP71: FIDUCIAL1X2, SparkFun-Aesthetics:FIDUCIAL-1X2
- removed JP33, JP36, JP39, JP42, JP45, JP48, JP51, JP54, JP57, JP60, JP63, JP66, JP69, JP72: USB_SOLDER_PADS, SparkFun-Connectors:USB-SOLDER-PADS
- removed L10, L11, L12, L13, L14, L15, L16, L17, L18, L19, L20, L21, L22, L23, L24, L7, L8, L9: 4.7μH, SparkFun-Coils:1008(2520)
- removed LED10, LED11, LED12, LED13, LED14, LED15, LED16, LED17, LED18, LED19, LED20, LED21, LED22, LED23, LED24, LED7, LED8, LED9: Red, SparkFun-LED:LED-0603
- removed LOGO19, LOGO22, LOGO25, LOGO28, LOGO31, LOGO34, LOGO37, LOGO40, LOGO43, LOGO46, LOGO49, LOGO52, LOGO55, LOGO58, LOGO61, LOGO64, LOGO67, LOGO70: SFE_LOGO_NAME_FLAME.1_INCH, SparkFun-Aesthetics:SFE_LOGO_NAME_FLAME_.1
- removed LOGO20, LOGO23, LOGO26, LOGO29, LOGO32, LOGO35, LOGO38, LOGO41, LOGO44, LOGO47, LOGO50, LOGO53, LOGO56, LOGO59, LOGO62, LOGO65, LOGO68, LOGO71: QWIIC_LOGO_6MM, SparkFun-Aesthetics:QWIIC_6MM
- removed LOGO21, LOGO24, LOGO27, LOGO30, LOGO33, LOGO36, LOGO39, LOGO42, LOGO45, LOGO48, LOGO51, LOGO54, LOGO57, LOGO60, LOGO63, LOGO66, LOGO69, LOGO72: SFE_LOGO_FLAME.1_INCH, SparkFun-Aesthetics:SFE_LOGO_FLAME_.1
- removed PWR10, PWR11, PWR12, PWR13, PWR14, PWR15, PWR16, PWR17, PWR18, PWR19, PWR20, PWR21, PWR22, PWR23, PWR6, PWR7, PWR8, PWR9, SHLD10, SHLD11, SHLD12, SHLD13, SHLD14, SHLD15, SHLD16, SHLD17, SHLD18, SHLD19, SHLD20, SHLD21, SHLD22, SHLD23, SHLD6, SHLD7, SHLD8, SHLD9: JUMPER-SMT_2_NC_TRACE_SILK, SparkFun-Jumpers:SMT-JUMPER_2_NC_TRACE_SILK
- removed R100, R111, R112, R123, R124, R135, R136, R147, R148, R159, R160, R171, R172, R183, R184, R195, R196, R207, R208, R219, R220, R231, R232, R243, R244, R255, R256, R267, R268, R279, R280, R87, R88, R99: 5.1k, SparkFun-Resistors:0402-TIGHT
- removed R101, R102, R113, R114, R125, R126, R137, R138, R149, R150, R161, R162, R173, R174, R185, R186, R197, R198, R209, R210, R221, R222, R233, R234, R245, R246, R257, R258, R269, R270, R281, R282, R89, R90: 2.2k, SparkFun-Resistors:0402-TIGHT
- removed R103, R107, R115, R119, R127, R131, R139, R143, R151, R155, R163, R167, R175, R179, R187, R191, R199, R203, R211, R215, R223, R227, R235, R239, R247, R251, R259, R263, R271, R275, R283, R287, R79, R83, R91, R95: 1k, SparkFun-Resistors:0402-TIGHT
- removed R104, R105, R116, R117, R128, R129, R140, R141, R152, R153, R164, R165, R176, R177, R188, R189, R200, R201, R212, R213, R224, R225, R236, R237, R248, R249, R260, R261, R272, R273, R284, R285, R80, R81, R92, R93: 27, SparkFun-Resistors:0402-TIGHT
- removed R106, R118, R130, R142, R154, R166, R178, R190, R202, R214, R226, R238, R250, R262, R274, R286, R82, R94: 10Ω, SparkFun-Resistors:0402-TIGHT
- removed R108, R110, R120, R122, R132, R134, R144, R146, R156, R158, R168, R170, R180, R182, R192, R194, R204, R206, R216, R218, R228, R230, R240, R242, R252, R254, R264, R266, R276, R278, R288, R84, R86, R96, R98: 10k, SparkFun-Resistors:0402-TIGHT
- removed R109, R121, R133, R145, R157, R169, R181, R193, R205, R217, R229, R241, R253, R265, R277, R85, R97: 4.7k, SparkFun-Resistors:0402-TIGHT
- removed S13, S15, S17, S19, S21, S23, S25, S27, S29, S31, S33, S35, S37, S39, S41, S43, S45, S47: Reset, SparkFun-Switches:TACTILE_SWITCH_SMD_4.6X2.8MM
- removed S14, S16, S18, S20, S22, S24, S26, S28, S30, S32, S34, S36, S38, S40, S42, S44, S46, S48: Boot, SparkFun-Switches:TACTILE_SWITCH_SMD_4.6X2.8MM
- removed TP25, TP26, TP27, TP28, TP29, TP30, TP31, TP32, TP33, TP34, TP35, TP36, TP37, TP38, TP39, TP40, TP41, TP42, TP43, TP44, TP45, TP46, TP47, TP48, TP49, TP50, TP51, TP52, TP53, TP54, TP55, TP56, TP57, TP58, TP59, TP60, TP61, TP62, TP63, TP64, TP65, TP66, TP67, TP68, TP69, TP70, TP71, TP72, TP73, TP74, TP75, TP76, TP77, TP78, TP79, TP80, TP81, TP82, TP83, TP84, TP85, TP86, TP87, TP88, TP89, TP90, TP91, TP92, TP93, TP94, TP95, TP96: TEST-POINT3X5, SparkFun-Connectors:PAD.03X.05
- removed U$1000, U$1058, U$1116, U$1174, U$1232, U$1290, U$1348, U$362, U$420, U$478, U$536, U$594, U$652, U$710, U$768, U$826, U$884, U$942: (no value), output:#RST#1
- removed U$1001, U$1059, U$1117, U$1175, U$1233, U$1291, U$1349, U$363, U$421, U$479, U$537, U$595, U$653, U$711, U$769, U$827, U$885, U$943: (no value), output:3V30
- removed U$1002, U$1060, U$1118, U$1176, U$1234, U$1292, U$1350, U$364, U$422, U$480, U$538, U$596, U$654, U$712, U$770, U$828, U$886, U$944: (no value), output:PWR0
- removed U$1003, U$1018, U$1031, U$1061, U$1076, U$1089, U$1119, U$1134, U$1147, U$1177, U$1192, U$1205, U$1235, U$1250, U$1263, U$1293, U$1308, U$1321, U$1351, U$1366, U$1379, U$365, U$380, U$393, U$423, U$438, U$451, U$481, U$496, U$509, U$539, U$554, U$567, U$597, U$612, U$625, U$655, U$670, U$683, U$713, U$728, U$741, U$771, U$786, U$799, U$829, U$844, U$857, U$887, U$902, U$915, U$945, U$960, U$973: (no value), output:GND2
- removed U$1004, U$1017, U$1062, U$1075, U$1120, U$1133, U$1178, U$1191, U$1236, U$1249, U$1294, U$1307, U$1352, U$1365, U$366, U$379, U$424, U$437, U$482, U$495, U$540, U$553, U$598, U$611, U$656, U$669, U$714, U$727, U$772, U$785, U$830, U$843, U$888, U$901, U$946, U$959: (no value), output:RX1
- removed U$1005, U$1016, U$1063, U$1074, U$1121, U$1132, U$1179, U$1190, U$1237, U$1248, U$1295, U$1306, U$1353, U$1364, U$367, U$378, U$425, U$436, U$483, U$494, U$541, U$552, U$599, U$610, U$657, U$668, U$715, U$726, U$773, U$784, U$831, U$842, U$889, U$900, U$947, U$958: (no value), output:TX0
- removed U$1006, U$1064, U$1122, U$1180, U$1238, U$1296, U$1354, U$368, U$426, U$484, U$542, U$600, U$658, U$716, U$774, U$832, U$890, U$948: (no value), output:GND_0
- removed U$1007, U$1065, U$1123, U$1181, U$1239, U$1297, U$1355, U$369, U$427, U$485, U$543, U$601, U$659, U$717, U$775, U$833, U$891, U$949: (no value), output:70
- removed U$1008, U$1066, U$1124, U$1182, U$1240, U$1298, U$1356, U$370, U$428, U$486, U$544, U$602, U$660, U$718, U$776, U$834, U$892, U$950: (no value), output:81
- removed U$1009, U$1067, U$1125, U$1183, U$1241, U$1299, U$1357, U$371, U$429, U$487, U$545, U$603, U$661, U$719, U$777, U$835, U$893, U$951: (no value), output:92
- removed U$1010, U$1050, U$1068, U$1108, U$1126, U$1166, U$1184, U$1224, U$1242, U$1282, U$1300, U$1340, U$1358, U$354, U$372, U$412, U$430, U$470, U$488, U$528, U$546, U$586, U$604, U$644, U$662, U$702, U$720, U$760, U$778, U$818, U$836, U$876, U$894, U$934, U$952, U$992: (no value), output:CI4
- removed U$1011, U$1052, U$1069, U$1110, U$1127, U$1168, U$1185, U$1226, U$1243, U$1284, U$1301, U$1342, U$1359, U$356, U$373, U$414, U$431, U$472, U$489, U$530, U$547, U$588, U$605, U$646, U$663, U$704, U$721, U$762, U$779, U$820, U$837, U$878, U$895, U$936, U$953, U$994: (no value), output:SCK3
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Connections:
- net QSPI-CS renamed FLASH_!CS!/BOOT
- removed net !RESET!10: J43.3, J43.3B, R122.1, S21.3, S21.4, U44.26
- removed net !RESET!11: J47.3, J47.3B, R134.1, S23.3, S23.4, U48.26
- removed net !RESET!12: J51.3, J51.3B, R146.1, S25.3, S25.4, U52.26
- removed net !RESET!13: J55.3, J55.3B, R158.1, S27.3, S27.4, U56.26
- removed net !RESET!14: J59.3, J59.3B, R170.1, S29.3, S29.4, U60.26
- removed net !RESET!15: J63.3, J63.3B, R182.1, S31.3, S31.4, U64.26
- removed net !RESET!16: J67.3, J67.3B, R194.1, S33.3, S33.4, U68.26
- removed net !RESET!17: J71.3, J71.3B, R206.1, S35.3, S35.4, U72.26
- removed net !RESET!18: J75.3, J75.3B, R218.1, S37.3, S37.4, U76.26
- removed net !RESET!19: J79.3, J79.3B, R230.1, S39.3, S39.4, U80.26
- removed net !RESET!20: J83.3, J83.3B, R242.1, S41.3, S41.4, U84.26
- removed net !RESET!21: J87.3, J87.3B, R254.1, S43.3, S43.4, U88.26
- removed net !RESET!22: J91.3, J91.3B, R266.1, S45.3, S45.4, U92.26
- removed net !RESET!23: J95.3, J95.3B, R278.1, S47.3, S47.4, U96.26
- removed net !RESET!6: J27.3, J27.3B, R74.1, S13.3, S13.4, U28.26
- removed net !RESET!7: J31.3, J31.3B, R86.1, S15.3, S15.4, U32.26
- removed net !RESET!8: J35.3, J35.3B, R98.1, S17.3, S17.4, U36.26
- removed net !RESET!9: J39.3, J39.3B, R110.1, S19.3, S19.4, U40.26
- removed net 0/TX10: J42.12, J42.12B, U44.2
- removed net 0/TX11: J46.12, J46.12B, U48.2
- removed net 0/TX12: J50.12, J50.12B, U52.2
- removed net 0/TX13: J54.12, J54.12B, U56.2
- removed net 0/TX14: J58.12, J58.12B, U60.2
- removed net 0/TX15: J62.12, J62.12B, U64.2
- removed net 0/TX16: J66.12, J66.12B, U68.2
- removed net 0/TX17: J70.12, J70.12B, U72.2
- removed net 0/TX18: J74.12, J74.12B, U76.2
- removed net 0/TX19: J78.12, J78.12B, U80.2
- removed net 0/TX20: J82.12, J82.12B, U84.2
- removed net 0/TX21: J86.12, J86.12B, U88.2
- removed net 0/TX22: J90.12, J90.12B, U92.2
- removed net 0/TX23: J94.12, J94.12B, U96.2
- removed net 0/TX6: J26.12, J26.12B, U28.2
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Routing:
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- removed copper zone on layer 1, net 1.1V10
- removed copper zone on layer 1, net 1.1V11
- removed copper zone on layer 1, net 1.1V12
- removed copper zone on layer 1, net 1.1V13
- removed copper zone on layer 1, net 1.1V14
- removed copper zone on layer 1, net 1.1V15
- removed copper zone on layer 1, net 1.1V16
- removed copper zone on layer 1, net 1.1V17
- removed copper zone on layer 1, net 1.1V18
- removed copper zone on layer 1, net 1.1V19
- removed copper zone on layer 1, net 1.1V20
- removed copper zone on layer 1, net 1.1V21
- removed copper zone on layer 1, net 1.1V22
- removed copper zone on layer 1, net 1.1V23
- removed copper zone on layer 1, net 1.1V6
- removed copper zone on layer 1, net 1.1V7
- removed copper zone on layer 1, net 1.1V8
- removed copper zone on layer 1, net 1.1V9
- removed copper zone on layer 1, net 3.3V10
- removed copper zone on layer 15, net 3.3V10
- removed copper zone on layer 1, net 3.3V11
- removed copper zone on layer 15, net 3.3V11
- removed copper zone on layer 1, net 3.3V12
- removed copper zone on layer 15, net 3.3V12
- removed copper zone on layer 1, net 3.3V13
- removed copper zone on layer 15, net 3.3V13
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Other:
- board size 207 x 125.5 mm -> 92.7 x 87.1 mm
- board text added: "v09"
- board text removed: "v10"

Commit message: Add v02 panel files
Parts:
- added U$349: (no value), output:B0
- added U$350: (no value), output:#SHLD#0
- added U$351: (no value), output:#P#0
- added U$352: (no value), output:BOOT0
- added U$353: (no value), output:RST0
- added U$354: (no value), output:RP23500
- U$100: device output:210 -> output:V3
- U$101: device output:#RST#0 -> output:210
- U$102: device output:3V3_0 -> output:#RST#0
- U$103: device output:GND2 -> output:3V3_0
- U$104: device output:RAW0 -> output:GND2
- U$105: device output:R0 -> output:RAW0
- U$106: device output:#0 -> output:R0
- U$107: device output:PRO_MICRO0 -> output:#0
- U$108: device output:C0 -> output:PRO_MICRO0
- U$109: device output:D1 -> output:C0
- U$110: device output:DO0 -> output:D1
- U$111: device output:RP23500 -> output:DO0
- U$112: device output:B0 -> output:RP23500
- U$113: device output:#SHLD#0 -> output:B0
- U$114: device output:#P#0 -> output:#SHLD#0
- U$115: device output:BOOT0 -> output:#P#0
- U$116: device output:RST0 -> output:BOOT0
- U$117: value OSHW-LOGOMINI -> (none); device SparkFun-Aesthetics:OSHW-LOGO-MINI -> output:RST0
- U$118: device output:A00 -> output:RP23500
- U$119: value (none) -> OSHW-LOGOMINI; device output:A10 -> SparkFun-Aesthetics:OSHW-LOGO-MINI
- U$120, U$144: device output:A21 -> output:A00
- U$121, U$145: device output:A32 -> output:A10
- U$122: device output:CI4 -> output:A21
- U$123: device output:CO5 -> output:A32
- U$124, U$83: device output:SCK3 -> output:CI4
- U$125: device output:20 -> output:CO5
- U$126: device output:31 -> output:SCK3
- U$127, U$151: device output:42 -> output:20
- U$128, U$152: device output:53 -> output:31
- U$129, U$153: device output:64 -> output:42
- U$130: device output:#RST#1 -> output:53
- U$131: device output:3V30 -> output:64
- U$132: device output:PWR0 -> output:#RST#1
- U$133: device output:GND2 -> output:3V30
- U$134: device output:RX1 -> output:PWR0
- U$135: device output:TX0 -> output:GND2
- U$136: device output:GND_0 -> output:RX1
- U$137: device output:70 -> output:TX0
- U$138: device output:81 -> output:GND_0
- U$139: device output:92 -> output:70
- U$140: device output:CI4 -> output:81
- U$141: device output:SCK3 -> output:92
- U$142: device output:A00 -> output:CI4
- U$143: device output:A10 -> output:SCK3
- U$146: device output:TX0 -> output:A21
- U$147: device output:RX1 -> output:A32
- U$148: device output:GND2 -> output:TX0
- U$149: device output:20 -> output:RX1
- U$150: device output:31 -> output:GND2
- U$154: device output:D#1 -> output:53
- U$155: device output:D#2 -> output:64
- U$156: device output:G0 -> output:D#1
- U$157: device output:V3 -> output:D#2
- U$158: device output:210 -> output:G0
- U$159: device output:#RST#0 -> output:V3
- U$160: device output:3V3_0 -> output:210
- U$161: device output:GND2 -> output:#RST#0
- U$162: device output:RAW0 -> output:3V3_0
- U$163: device output:R0 -> output:GND2
- U$164: device output:#0 -> output:RAW0
- U$165: device output:PRO_MICRO0 -> output:R0
- U$166: device output:C0 -> output:#0
- U$167: device output:D1 -> output:PRO_MICRO0
- U$168: device output:DO0 -> output:C0
- U$169: device output:RP23500 -> output:D1
- U$170: device output:B0 -> output:DO0
- U$171: device output:#SHLD#0 -> output:RP23500
- U$172: device output:#P#0 -> output:B0
- U$173: device output:BOOT0 -> output:#SHLD#0
- U$174: device output:RST0 -> output:#P#0
- U$175: value OSHW-LOGOMINI -> (none); device SparkFun-Aesthetics:OSHW-LOGO-MINI -> output:BOOT0
- U$176: device output:A00 -> output:RST0
- U$177: device output:A10 -> output:RP23500
- U$178: value (none) -> OSHW-LOGOMINI; device output:A21 -> SparkFun-Aesthetics:OSHW-LOGO-MINI
- U$179, U$203: device output:A32 -> output:A00
- U$180: device output:CI4 -> output:A10
- U$181: device output:CO5 -> output:A21
- U$182: device output:SCK3 -> output:A32
- U$183: device output:20 -> output:CI4
- U$184: device output:31 -> output:CO5
- U$185: device output:42 -> output:SCK3
- U$186, U$210: device output:53 -> output:20
- U$187, U$211: device output:64 -> output:31
- U$188: device output:#RST#1 -> output:42
- U$189: device output:3V30 -> output:53
- U$190: device output:PWR0 -> output:64
- U$191: device output:GND2 -> output:#RST#1
- U$192: device output:RX1 -> output:3V30
- U$193: device output:TX0 -> output:PWR0
- U$194: device output:GND_0 -> output:GND2
- U$195: device output:70 -> output:RX1
- U$196: device output:81 -> output:TX0
- U$197: device output:92 -> output:GND_0
- U$198: device output:CI4 -> output:70
- U$199: device output:SCK3 -> output:81
- U$200: device output:A00 -> output:92
- U$201: device output:A10 -> output:CI4
- U$202: device output:A21 -> output:SCK3
- U$204: device output:TX0 -> output:A10
- U$205: device output:RX1 -> output:A21
- U$206: device output:GND2 -> output:A32
- U$207: device output:20 -> output:TX0
- U$208: device output:31 -> output:RX1
- U$209: device output:42 -> output:GND2
- U$212: device output:D#1 -> output:42
- U$213: device output:D#2 -> output:53
- U$214: device output:G0 -> output:64
- U$215: device output:V3 -> output:D#1
- U$216: device output:210 -> output:D#2
- U$217: device output:#RST#0 -> output:G0
- U$218: device output:3V3_0 -> output:V3
- U$219: device output:GND2 -> output:210
- U$220: device output:RAW0 -> output:#RST#0
- U$221: device output:R0 -> output:3V3_0
- U$222: device output:#0 -> output:GND2
- U$223: device output:PRO_MICRO0 -> output:RAW0
- U$224: device output:C0 -> output:R0
- U$225: device output:D1 -> output:#0
- U$226: device output:DO0 -> output:PRO_MICRO0
- U$227: device output:RP23500 -> output:C0
- U$228: device output:B0 -> output:D1
- U$229: device output:#SHLD#0 -> output:DO0
- U$230: device output:#P#0 -> output:RP23500
- U$231: device output:BOOT0 -> output:B0
- U$232: device output:RST0 -> output:#SHLD#0
- U$233: value OSHW-LOGOMINI -> (none); device SparkFun-Aesthetics:OSHW-LOGO-MINI -> output:#P#0
- U$234: device output:A00 -> output:BOOT0
- U$235: device output:A10 -> output:RST0
- U$236: device output:A21 -> output:RP23500
- U$237: value (none) -> OSHW-LOGOMINI; device output:A32 -> SparkFun-Aesthetics:OSHW-LOGO-MINI
- U$238: device output:CI4 -> output:A00
- U$239: device output:CO5 -> output:A10
- U$240: device output:SCK3 -> output:A21
- U$241, U$265: device output:20 -> output:A32
- U$242: device output:31 -> output:CI4
- U$243: device output:42 -> output:CO5
- U$244: device output:53 -> output:SCK3
- U$245, U$269: device output:64 -> output:20
- U$246: device output:#RST#1 -> output:31
- U$247: device output:3V30 -> output:42
- U$248: device output:PWR0 -> output:53
- U$249: device output:GND2 -> output:64
- U$250: device output:RX1 -> output:#RST#1
- U$251: device output:TX0 -> output:3V30
- U$252: device output:GND_0 -> output:PWR0
- U$253: device output:70 -> output:GND2
- U$254: device output:81 -> output:RX1
- U$255: device output:92 -> output:TX0
- U$256: device output:CI4 -> output:GND_0
- U$257: device output:SCK3 -> output:70
- U$258: device output:A00 -> output:81
- U$259: device output:A10 -> output:92
- U$260: device output:A21 -> output:CI4
- U$261: device output:A32 -> output:SCK3
- U$262: device output:TX0 -> output:A00
- U$263: device output:RX1 -> output:A10
- U$264: device output:GND2 -> output:A21
- U$266: device output:31 -> output:TX0
- U$267: device output:42 -> output:RX1
- U$268: device output:53 -> output:GND2
- U$270: device output:D#1 -> output:31
- U$271: device output:D#2 -> output:42
- U$272: device output:G0 -> output:53
- U$273: device output:V3 -> output:64
- U$274: device output:210 -> output:D#1
- U$275: device output:#RST#0 -> output:D#2
- U$276: device output:3V3_0 -> output:G0
- U$277: device output:GND2 -> output:V3
- U$278: device output:RAW0 -> output:210
- U$279: device output:R0 -> output:#RST#0
- U$280: device output:#0 -> output:3V3_0
- U$281: device output:PRO_MICRO0 -> output:GND2
- U$282: device output:C0 -> output:RAW0
- U$283: device output:D1 -> output:R0
- U$284: device output:DO0 -> output:#0
- U$285: device output:RP23500 -> output:PRO_MICRO0
- U$286: device output:B0 -> output:C0
- U$287: device output:#SHLD#0 -> output:D1
- U$288: device output:#P#0 -> output:DO0
- U$289: device output:BOOT0 -> output:RP23500
- U$290: device output:RST0 -> output:B0
- U$291: value OSHW-LOGOMINI -> (none); device SparkFun-Aesthetics:OSHW-LOGO-MINI -> output:#SHLD#0
- U$292: device output:A00 -> output:#P#0
- U$293: device output:A10 -> output:BOOT0
- U$294: device output:A21 -> output:RST0
- U$295: device output:A32 -> output:RP23500
- U$296: value (none) -> OSHW-LOGOMINI; device output:CI4 -> SparkFun-Aesthetics:OSHW-LOGO-MINI
- U$297: device output:CO5 -> output:A00
- U$298: device output:SCK3 -> output:A10
- U$299, U$323: device output:20 -> output:A21
- U$300, U$324: device output:31 -> output:A32
- U$301: device output:42 -> output:CI4
- U$302: device output:53 -> output:CO5
- U$303: device output:64 -> output:SCK3
- U$304: device output:#RST#1 -> output:20
- U$305: device output:3V30 -> output:31
- U$306: device output:PWR0 -> output:42
- U$307: device output:GND2 -> output:53
- U$308: device output:RX1 -> output:64
- U$309: device output:TX0 -> output:#RST#1
- U$310: device output:GND_0 -> output:3V30
- U$311: device output:70 -> output:PWR0
- U$312: device output:81 -> output:GND2
- U$313: device output:92 -> output:RX1
- U$314: device output:CI4 -> output:TX0
- U$315: device output:SCK3 -> output:GND_0
- U$316: device output:A00 -> output:70
- U$317: device output:A10 -> output:81
- U$318: device output:A21 -> output:92
- U$319: device output:A32 -> output:CI4
- U$320: device output:TX0 -> output:SCK3
- U$321: device output:RX1 -> output:A00
- U$322: device output:GND2 -> output:A10
- U$325: device output:42 -> output:TX0
- U$326: device output:53 -> output:RX1
- U$327: device output:64 -> output:GND2
- U$328: device output:D#1 -> output:20
- U$329: device output:D#2 -> output:31
- U$330: device output:G0 -> output:42
- U$331: device output:V3 -> output:53
- U$332: device output:210 -> output:64
- U$333: device output:#RST#0 -> output:D#1
- U$334: device output:3V3_0 -> output:D#2
- U$335: device output:GND2 -> output:G0
- U$336: device output:RAW0 -> output:V3
- U$337: device output:R0 -> output:210
- U$338: device output:#0 -> output:#RST#0
- U$339: device output:PRO_MICRO0 -> output:3V3_0
- U$340: device output:C0 -> output:GND2
- U$341: device output:D1 -> output:RAW0
- U$342: device output:DO0 -> output:R0
- U$343: device output:RP23500 -> output:#0
- U$344: device output:B0 -> output:PRO_MICRO0
- U$345: device output:#SHLD#0 -> output:C0
- U$346: device output:#P#0 -> output:D1
- U$347: device output:BOOT0 -> output:DO0
- U$348: device output:RST0 -> output:RP23500
- U$45: value OSHW-LOGOMINI -> (none); device SparkFun-Aesthetics:OSHW-LOGO-MINI -> output:RP23500
- U$46: value (none) -> OSHW-LOGOMINI; device output:A00 -> SparkFun-Aesthetics:OSHW-LOGO-MINI
- U$47, U$85: device output:A10 -> output:A00
- U$48, U$86: device output:A21 -> output:A10
- U$49, U$87: device output:A32 -> output:A21
- U$50: device output:CI4 -> output:A32
- U$51: device output:CO5 -> output:CI4
- U$52: device output:SCK3 -> output:CO5
- U$58: device output:20 -> output:SCK3
- U$59, U$92: device output:31 -> output:20
- U$60, U$93: device output:42 -> output:31
- U$61, U$94: device output:53 -> output:42
- U$62, U$95: device output:64 -> output:53
- U$63: device output:#RST#1 -> output:64
- U$65: device output:3V30 -> output:#RST#1
- U$70: device output:PWR0 -> output:3V30
- U$71: device output:GND2 -> output:PWR0
- U$72: device output:RX1 -> output:GND2
- U$77: device output:TX0 -> output:RX1
- U$78: device output:GND_0 -> output:TX0
- U$79: device output:70 -> output:GND_0
- U$80: device output:81 -> output:70
- U$81: device output:92 -> output:81
- U$82: device output:CI4 -> output:92
- U$84: device output:A00 -> output:SCK3
- U$88: device output:TX0 -> output:A32
- U$89: device output:RX1 -> output:TX0
- U$90: device output:GND2 -> output:RX1
- U$91: device output:20 -> output:GND2
- U$96: device output:D#1 -> output:64
- U$97: device output:D#2 -> output:D#1
- U$98: device output:G0 -> output:D#2
- U$99: device output:V3 -> output:G0
- moved U$175 66.2 mm to (51.3, 2.54), turned to 0 degrees
- moved U$176 65.1 mm to (57.7, 2.54), flipped to the bottom, turned to 0 degrees
- moved U$177 49.7 mm to (54.6, 24.1), turned to 0 degrees
- moved U$292 39.5 mm to (26.2, 70.7), flipped to the bottom, turned to 0 degrees
- moved U$293 34.3 mm to (28.4, 42.9), flipped to the bottom, turned to 0 degrees
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Routing:
- net 16/SDA2: track 12.0 -> 4.69 mm, vias 2 -> 0
- net 16/SDA5: track 12.0 -> 4.69 mm, vias 2 -> 0
- net 16/SDA: track 12.0 -> 4.69 mm, vias 2 -> 0
- net 16/SDA3: track 12.0 -> 4.69 mm, vias 2 -> 0
- net 16/SDA1: track 12.0 -> 4.69 mm, vias 2 -> 0
- net 16/SDA4: track 12.0 -> 4.69 mm, vias 2 -> 0
- net 17/SCL5: track 10.7 -> 4.62 mm, vias 2 -> 0
- net 17/SCL2: track 10.7 -> 4.62 mm, vias 2 -> 0
- net 17/SCL3: track 10.7 -> 4.62 mm, vias 2 -> 0
- net 17/SCL: track 10.7 -> 4.62 mm, vias 2 -> 0
- net 17/SCL4: track 10.7 -> 4.62 mm, vias 2 -> 0
- net 17/SCL1: track 10.7 -> 4.62 mm, vias 2 -> 0
- net N$4: track 7.29 -> 1.72 mm, vias 2 -> 0
- net N$11: track 7.29 -> 1.72 mm, vias 2 -> 0
- net N$9: track 7.29 -> 1.72 mm, vias 2 -> 0
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Other:
- board text added: "v02"
- board text removed: "v09"
