File: Production/SparkFun_ProMicro_RP2350-Panel.brd (EAGLE design)
At the start: 92.7 x 87.1 mm, 738 parts, among them J1 QWIIC_RIGHT_ANGLE, J12 USB Female Type C Connector, J13 QWIIC_RIGHT_ANGLE, J16 USB Female Type C Connector, J17 QWIIC_RIGHT_ANGLE, J2 QWIIC_RIGHT_ANGLE, J20 USB Female Type C Connector, J21 QWIIC_RIGHT_ANGLE, J24 USB Female Type C Connector, J5 USB Female Type C Connector, J8 USB Female Type C Connector, J9 QWIIC_RIGHT_ANGLE, U1 RT9080-33GJ5, U10 APS6404L-3SQR-ZR, U11 RT9080-33GJ5, U12 W25QXX128MBIT, U13 WS2812_2020, U14 RP2350A, U15 APS6404L-3SQR-ZR, U16 RT9080-33GJ5, U17 W25QXX128MBIT, U18 WS2812_2020, U19 RP2350A, U2 RP2350A, U20 APS6404L-3SQR-ZR, U21 RT9080-33GJ5, U22 W25QXX128MBIT, U23 WS2812_2020, U24 RP2350A, U25 APS6404L-3SQR-ZR, U26 RT9080-33GJ5, U27 W25QXX128MBIT, U28 WS2812_2020, U29 RP2350A, U3 WS2812_2020, U30 APS6404L-3SQR-ZR, U4 W25QXX128MBIT, U5 APS6404L-3SQR-ZR, U6 RT9080-33GJ5, U7 W25QXX128MBIT, U8 WS2812_2020, U9 RP2350A, Y1 12MHz, Y2 12MHz, Y3 12MHz, Y4 12MHz, Y5 12MHz, Y6 12MHz

Commit message: Add v10 production files
Parts:
- added C121, C122, C133, C134, C141, C142, C153, C154, C161, C162, C173, C174, C181, C182, C193, C194, C201, C202, C213, C214, C221, C222, C233, C234, C241, C242, C253, C254, C261, C262, C273, C274, C281, C282, C293, C294, C301, C302, C313, C314, C321, C322, C333, C334, C341, C342, C353, C354, C361, C362, C373, C374, C381, C382, C393, C394, C401, C402, C413, C414, C421, C422, C433, C434, C441, C442, C453, C454, C461, C462, C473, C474: 10uF, SparkFun-Capacitors:0402-TIGHT
- added C123, C124, C143, C144, C163, C164, C183, C184, C203, C204, C223, C224, C243, C244, C263, C264, C283, C284, C303, C304, C323, C324, C343, C344, C363, C364, C383, C384, C403, C404, C423, C424, C443, C444, C463, C464: 15pF, SparkFun-Capacitors:0402-TIGHT
- added C125, C126, C127, C128, C129, C130, C131, C132, C136, C138, C139, C140, C145, C146, C147, C148, C149, C150, C151, C152, C156, C158, C159, C160, C165, C166, C167, C168, C169, C170, C171, C172, C176, C178, C179, C180, C185, C186, C187, C188, C189, C190, C191, C192, C196, C198, C199, C200, C205, C206, C207, C208, C209, C210, C211, C212, C216, C218, C219, C220, C225, C226, C227, C228, C229, C230, C231, C232, C236, C238, C239, C240, C245, C246, C247, C248, C249, C250, C251, C252, C256, C258, C259, C260, C265, C266, C267, C268, C269, C270, C271, C272, C276, C278, C279, C280, C285, C286, C287, C288, C289, C290, C291, C292, C296, C298, C299, C300, C305, C306, C307, C308, C309, C310, C311, C312, C316, C318, C319, C320, C325, C326, C327, C328, C329, C330, C331, C332, C336, C338, C339, C340, C345, C346, C347, C348, C349, C350, C351, C352, C356, C358, C359, C360, C365, C366, C367, C368, C369, C370, C371, C372, C376, C378, C379, C380, C385, C386, C387, C388, C389, C390, C391, C392, C396, C398, C399, C400, C405, C406, C407, C408, C409, C410, C411, C412, C416, C418, C419, C420, C425, C426, C427, C428, C429, C430, C431, C432, C436, C438, C439, C440, C445, C446, C447, C448, C449, C450, C451, C452, C456, C458, C459, C460, C465, C466, C467, C468, C469, C470, C471, C472, C476, C478, C479, C480: 0.1uF, SparkFun-Capacitors:0402-TIGHT
- added C135, C137, C155, C157, C175, C177, C195, C197, C215, C217, C235, C237, C255, C257, C275, C277, C295, C297, C315, C317, C335, C337, C355, C357, C375, C377, C395, C397, C415, C417, C435, C437, C455, C457, C475, C477: 2.2uF, SparkFun-Capacitors:0402-TIGHT
- added D10, D11, D12, D13, D14, D15, D16, D17, D18, D19, D20, D21, D22, D23, D24, D7, D8, D9: 3A/10V/280mV, SparkFun-DiscreteSemi:SOD-323
- added F10, F11, F12, F13, F14, F15, F16, F17, F18, F19, F20, F21, F22, F23, F24, F7, F8, F9: 6V 0.5A, SparkFun-Fuses:0805
- added J25, J29, J33, J37, J41, J45, J49, J53, J57, J61, J65, J69, J73, J77, J81, J85, J89, J93: QWIIC_RIGHT_ANGLE, SparkFun-Connectors:JST04_1MM_RA
- added J26, J27, J30, J31, J34, J35, J38, J39, J42, J43, J46, J47, J50, J51, J54, J55, J58, J59, J62, J63, J66, J67, J70, J71, J74, J75, J78, J79, J82, J83, J86, J87, J90, J91, J94, J95: (no value), SparkFun-Connectors:1X12_CASTELLATED
- added J28, J32, J36, J40, J44, J48, J52, J56, J60, J64, J68, J72, J76, J80, J84, J88, J92, J96: USB Female Type C Connector, SparkFun-Connectors:USB-C-16P_4LAYER-PADS
- added JP100, JP101, JP102, JP104, JP105, JP106, JP107, JP109, JP110, JP111, JP112, JP114, JP115, JP116, JP117, JP119, JP120, JP31, JP32, JP34, JP35, JP36, JP37, JP39, JP40, JP41, JP42, JP44, JP45, JP46, JP47, JP49, JP50, JP51, JP52, JP54, JP55, JP56, JP57, JP59, JP60, JP61, JP62, JP64, JP65, JP66, JP67, JP69, JP70, JP71, JP72, JP74, JP75, JP76, JP77, JP79, JP80, JP81, JP82, JP84, JP85, JP86, JP87, JP89, JP90, JP91, JP92, JP94, JP95, JP96, JP97, JP99: FIDUCIAL1X2, SparkFun-Aesthetics:FIDUCIAL-1X2
- added JP103, JP108, JP113, JP118, JP33, JP38, JP43, JP48, JP53, JP58, JP63, JP68, JP73, JP78, JP83, JP88, JP93, JP98: USB_SOLDER_PADS, SparkFun-Connectors:USB-SOLDER-PADS
- added L10, L11, L12, L13, L14, L15, L16, L17, L18, L19, L20, L21, L22, L23, L24, L7, L8, L9: 4.7μH, SparkFun-Coils:1008(2520)
- added LED10, LED11, LED12, LED13, LED14, LED15, LED16, LED17, LED18, LED19, LED20, LED21, LED22, LED23, LED24, LED7, LED8, LED9: Red, SparkFun-LED:LED-0603
- added LOGO19, LOGO22, LOGO25, LOGO28, LOGO31, LOGO34, LOGO37, LOGO40, LOGO43, LOGO46, LOGO49, LOGO52, LOGO55, LOGO58, LOGO61, LOGO64, LOGO67, LOGO70: SFE_LOGO_NAME_FLAME.1_INCH, SparkFun-Aesthetics:SFE_LOGO_NAME_FLAME_.1
- added LOGO20, LOGO23, LOGO26, LOGO29, LOGO32, LOGO35, LOGO38, LOGO41, LOGO44, LOGO47, LOGO50, LOGO53, LOGO56, LOGO59, LOGO62, LOGO65, LOGO68, LOGO71: QWIIC_LOGO_6MM, SparkFun-Aesthetics:QWIIC_6MM
- added LOGO21, LOGO24, LOGO27, LOGO30, LOGO33, LOGO36, LOGO39, LOGO42, LOGO45, LOGO48, LOGO51, LOGO54, LOGO57, LOGO60, LOGO63, LOGO66, LOGO69, LOGO72: SFE_LOGO_FLAME.1_INCH, SparkFun-Aesthetics:SFE_LOGO_FLAME_.1
- added PWR10, PWR11, PWR12, PWR13, PWR14, PWR15, PWR16, PWR17, PWR18, PWR19, PWR20, PWR21, PWR22, PWR23, PWR6, PWR7, PWR8, PWR9, SHLD10, SHLD11, SHLD12, SHLD13, SHLD14, SHLD15, SHLD16, SHLD17, SHLD18, SHLD19, SHLD20, SHLD21, SHLD22, SHLD23, SHLD6, SHLD7, SHLD8, SHLD9: JUMPER-SMT_2_NC_TRACE_SILK, SparkFun-Jumpers:SMT-JUMPER_2_NC_TRACE_SILK
- added R100, R112, R113, R125, R126, R138, R139, R151, R152, R164, R165, R177, R178, R190, R191, R203, R204, R216, R217, R229, R230, R242, R243, R255, R256, R268, R269, R281, R282, R294, R295, R307, R308, R86, R87, R99: 27, SparkFun-Resistors:0402-TIGHT
- added R101, R114, R127, R140, R153, R166, R179, R192, R205, R218, R231, R244, R257, R270, R283, R296, R309, R88: 10Ω, SparkFun-Resistors:0402-TIGHT
- added R102, R111, R115, R124, R128, R137, R141, R150, R154, R163, R167, R176, R180, R189, R193, R202, R206, R215, R219, R228, R232, R241, R245, R254, R258, R267, R271, R280, R284, R293, R297, R306, R310, R85, R89, R98: 1k, SparkFun-Resistors:0402-TIGHT
- added R103, R104, R106, R116, R117, R119, R129, R130, R132, R142, R143, R145, R155, R156, R158, R168, R169, R171, R181, R182, R184, R194, R195, R197, R207, R208, R210, R220, R221, R223, R233, R234, R236, R246, R247, R249, R259, R260, R262, R272, R273, R275, R285, R286, R288, R298, R299, R301, R311, R312, R80, R90, R91, R93: 10k, SparkFun-Resistors:0402-TIGHT
- added R105, R118, R131, R144, R157, R170, R183, R196, R209, R222, R235, R248, R261, R274, R287, R300, R79, R92: 4.7k, SparkFun-Resistors:0402-TIGHT
- added R107, R108, R120, R121, R133, R134, R146, R147, R159, R160, R172, R173, R185, R186, R198, R199, R211, R212, R224, R225, R237, R238, R250, R251, R263, R264, R276, R277, R289, R290, R302, R303, R81, R82, R94, R95: 5.1k, SparkFun-Resistors:0402-TIGHT
- added R109, R110, R122, R123, R135, R136, R148, R149, R161, R162, R174, R175, R187, R188, R200, R201, R213, R214, R226, R227, R239, R240, R252, R253, R265, R266, R278, R279, R291, R292, R304, R305, R83, R84, R96, R97: 2.2k, SparkFun-Resistors:0402-TIGHT
- added S13, S15, S17, S19, S21, S23, S25, S27, S29, S31, S33, S35, S37, S39, S41, S43, S45, S47: Reset, SparkFun-Switches:TACTILE_SWITCH_SMD_4.6X2.8MM
- added S14, S16, S18, S20, S22, S24, S26, S28, S30, S32, S34, S36, S38, S40, S42, S44, S46, S48: Boot, SparkFun-Switches:TACTILE_SWITCH_SMD_4.6X2.8MM
- added TP25, TP26, TP27, TP28, TP29, TP30, TP31, TP32, TP33, TP34, TP35, TP36, TP37, TP38, TP39, TP40, TP41, TP42, TP43, TP44, TP45, TP46, TP47, TP48, TP49, TP50, TP51, TP52, TP53, TP54, TP55, TP56, TP57, TP58, TP59, TP60, TP61, TP62, TP63, TP64, TP65, TP66, TP67, TP68, TP69, TP70, TP71, TP72, TP73, TP74, TP75, TP76, TP77, TP78, TP79, TP80, TP81, TP82, TP83, TP84, TP85, TP86, TP87, TP88, TP89, TP90, TP91, TP92, TP93, TP94, TP95, TP96: TEST-POINT3X5, SparkFun-Connectors:PAD.03X.05
- added U$1000, U$1059, U$1118, U$1177, U$1236, U$1295, U$1354, U$1413, U$410, U$469, U$528, U$587, U$646, U$705, U$764, U$823, U$882, U$941: (no value), output:#P#0
- added U$1001, U$1060, U$1119, U$1178, U$1237, U$1296, U$1355, U$1414, U$411, U$470, U$529, U$588, U$647, U$706, U$765, U$824, U$883, U$942: (no value), output:BOOT0
- added U$1002, U$1061, U$1120, U$1179, U$1238, U$1297, U$1356, U$1415, U$412, U$471, U$530, U$589, U$648, U$707, U$766, U$825, U$884, U$943: (no value), output:RST0
- added U$1003, U$1056, U$1062, U$1115, U$1121, U$1174, U$1180, U$1233, U$1239, U$1292, U$1298, U$1351, U$1357, U$1410, U$1416, U$407, U$413, U$466, U$472, U$525, U$531, U$584, U$590, U$643, U$649, U$702, U$708, U$761, U$767, U$820, U$826, U$879, U$885, U$938, U$944, U$997: (no value), output:RP23500
- added U$1004, U$1063, U$1122, U$1181, U$1240, U$1299, U$1358, U$355, U$414, U$473, U$532, U$591, U$650, U$709, U$768, U$827, U$886, U$945: OSHW-LOGOMINI, SparkFun-Aesthetics:OSHW-LOGO-MINI
- added U$1005, U$1029, U$1064, U$1088, U$1123, U$1147, U$1182, U$1206, U$1241, U$1265, U$1300, U$1324, U$1359, U$1383, U$356, U$380, U$415, U$439, U$474, U$498, U$533, U$557, U$592, U$616, U$651, U$675, U$710, U$734, U$769, U$793, U$828, U$852, U$887, U$911, U$946, U$970: (no value), output:A00
- added U$1006, U$1030, U$1065, U$1089, U$1124, U$1148, U$1183, U$1207, U$1242, U$1266, U$1301, U$1325, U$1360, U$1384, U$357, U$381, U$416, U$440, U$475, U$499, U$534, U$558, U$593, U$617, U$652, U$676, U$711, U$735, U$770, U$794, U$829, U$853, U$888, U$912, U$947, U$971: (no value), output:A10
- added U$1007, U$1031, U$1066, U$1090, U$1125, U$1149, U$1184, U$1208, U$1243, U$1267, U$1302, U$1326, U$1361, U$1385, U$358, U$382, U$417, U$441, U$476, U$500, U$535, U$559, U$594, U$618, U$653, U$677, U$712, U$736, U$771, U$795, U$830, U$854, U$889, U$913, U$948, U$972: (no value), output:A21
- added U$1008, U$1032, U$1067, U$1091, U$1126, U$1150, U$1185, U$1209, U$1244, U$1268, U$1303, U$1327, U$1362, U$1386, U$359, U$383, U$418, U$442, U$477, U$501, U$536, U$560, U$595, U$619, U$654, U$678, U$713, U$737, U$772, U$796, U$831, U$855, U$890, U$914, U$949, U$973: (no value), output:A32
- added U$1009, U$1027, U$1068, U$1086, U$1127, U$1145, U$1186, U$1204, U$1245, U$1263, U$1304, U$1322, U$1363, U$1381, U$360, U$378, U$419, U$437, U$478, U$496, U$537, U$555, U$596, U$614, U$655, U$673, U$714, U$732, U$773, U$791, U$832, U$850, U$891, U$909, U$950, U$968: (no value), output:CI4
- added U$1010, U$1069, U$1128, U$1187, U$1246, U$1305, U$1364, U$361, U$420, U$479, U$538, U$597, U$656, U$715, U$774, U$833, U$892, U$951: (no value), output:CO5
- added U$1011, U$1028, U$1070, U$1087, U$1129, U$1146, U$1188, U$1205, U$1247, U$1264, U$1306, U$1323, U$1365, U$1382, U$362, U$379, U$421, U$438, U$480, U$497, U$539, U$556, U$598, U$615, U$657, U$674, U$716, U$733, U$775, U$792, U$834, U$851, U$893, U$910, U$952, U$969: (no value), output:SCK3
- added U$1012, U$1036, U$1071, U$1095, U$1130, U$1154, U$1189, U$1213, U$1248, U$1272, U$1307, U$1331, U$1366, U$1390, U$363, U$387, U$422, U$446, U$481, U$505, U$540, U$564, U$599, U$623, U$658, U$682, U$717, U$741, U$776, U$800, U$835, U$859, U$894, U$918, U$953, U$977: (no value), output:20
- added U$1013, U$1037, U$1072, U$1096, U$1131, U$1155, U$1190, U$1214, U$1249, U$1273, U$1308, U$1332, U$1367, U$1391, U$364, U$388, U$423, U$447, U$482, U$506, U$541, U$565, U$600, U$624, U$659, U$683, U$718, U$742, U$777, U$801, U$836, U$860, U$895, U$919, U$954, U$978: (no value), output:31
- added U$1014, U$1038, U$1073, U$1097, U$1132, U$1156, U$1191, U$1215, U$1250, U$1274, U$1309, U$1333, U$1368, U$1392, U$365, U$389, U$424, U$448, U$483, U$507, U$542, U$566, U$601, U$625, U$660, U$684, U$719, U$743, U$778, U$802, U$837, U$861, U$896, U$920, U$955, U$979: (no value), output:42
- added U$1015, U$1039, U$1074, U$1098, U$1133, U$1157, U$1192, U$1216, U$1251, U$1275, U$1310, U$1334, U$1369, U$1393, U$366, U$390, U$425, U$449, U$484, U$508, U$543, U$567, U$602, U$626, U$661, U$685, U$720, U$744, U$779, U$803, U$838, U$862, U$897, U$921, U$956, U$980: (no value), output:53
- added U$1016, U$1040, U$1075, U$1099, U$1134, U$1158, U$1193, U$1217, U$1252, U$1276, U$1311, U$1335, U$1370, U$1394, U$367, U$391, U$426, U$450, U$485, U$509, U$544, U$568, U$603, U$627, U$662, U$686, U$721, U$745, U$780, U$804, U$839, U$863, U$898, U$922, U$957, U$981: (no value), output:64
- added U$1017, U$1076, U$1135, U$1194, U$1253, U$1312, U$1371, U$368, U$427, U$486, U$545, U$604, U$663, U$722, U$781, U$840, U$899, U$958: (no value), output:#RST#1
- added U$1018, U$1077, U$1136, U$1195, U$1254, U$1313, U$1372, U$369, U$428, U$487, U$546, U$605, U$664, U$723, U$782, U$841, U$900, U$959: (no value), output:3V30
- added U$1019, U$1078, U$1137, U$1196, U$1255, U$1314, U$1373, U$370, U$429, U$488, U$547, U$606, U$665, U$724, U$783, U$842, U$901, U$960: (no value), output:PWR0
- added U$1020, U$1035, U$1048, U$1079, U$1094, U$1107, U$1138, U$1153, U$1166, U$1197, U$1212, U$1225, U$1256, U$1271, U$1284, U$1315, U$1330, U$1343, U$1374, U$1389, U$1402, U$371, U$386, U$399, U$430, U$445, U$458, U$489, U$504, U$517, U$548, U$563, U$576, U$607, U$622, U$635, U$666, U$681, U$694, U$725, U$740, U$753, U$784, U$799, U$812, U$843, U$858, U$871, U$902, U$917, U$930, U$961, U$976, U$989: (no value), output:GND2
- added U$1021, U$1034, U$1080, U$1093, U$1139, U$1152, U$1198, U$1211, U$1257, U$1270, U$1316, U$1329, U$1375, U$1388, U$372, U$385, U$431, U$444, U$490, U$503, U$549, U$562, U$608, U$621, U$667, U$680, U$726, U$739, U$785, U$798, U$844, U$857, U$903, U$916, U$962, U$975: (no value), output:RX1
- added U$1022, U$1033, U$1081, U$1092, U$1140, U$1151, U$1199, U$1210, U$1258, U$1269, U$1317, U$1328, U$1376, U$1387, U$373, U$384, U$432, U$443, U$491, U$502, U$550, U$561, U$609, U$620, U$668, U$679, U$727, U$738, U$786, U$797, U$845, U$856, U$904, U$915, U$963, U$974: (no value), output:TX0
- added U$1023, U$1082, U$1141, U$1200, U$1259, U$1318, U$1377, U$374, U$433, U$492, U$551, U$610, U$669, U$728, U$787, U$846, U$905, U$964: (no value), output:GND_0
- added U$1024, U$1083, U$1142, U$1201, U$1260, U$1319, U$1378, U$375, U$434, U$493, U$552, U$611, U$670, U$729, U$788, U$847, U$906, U$965: (no value), output:70
- added U$1025, U$1084, U$1143, U$1202, U$1261, U$1320, U$1379, U$376, U$435, U$494, U$553, U$612, U$671, U$730, U$789, U$848, U$907, U$966: (no value), output:81
- added U$1026, U$1085, U$1144, U$1203, U$1262, U$1321, U$1380, U$377, U$436, U$495, U$554, U$613, U$672, U$731, U$790, U$849, U$908, U$967: (no value), output:92
- added U$1041, U$1100, U$1159, U$1218, U$1277, U$1336, U$1395, U$392, U$451, U$510, U$569, U$628, U$687, U$746, U$805, U$864, U$923, U$982: (no value), output:D#1
- added U$1042, U$1101, U$1160, U$1219, U$1278, U$1337, U$1396, U$393, U$452, U$511, U$570, U$629, U$688, U$747, U$806, U$865, U$924, U$983: (no value), output:D#2
- added U$1043, U$1102, U$1161, U$1220, U$1279, U$1338, U$1397, U$394, U$453, U$512, U$571, U$630, U$689, U$748, U$807, U$866, U$925, U$984: (no value), output:G0
- added U$1044, U$1103, U$1162, U$1221, U$1280, U$1339, U$1398, U$395, U$454, U$513, U$572, U$631, U$690, U$749, U$808, U$867, U$926, U$985: (no value), output:V3
- added U$1045, U$1104, U$1163, U$1222, U$1281, U$1340, U$1399, U$396, U$455, U$514, U$573, U$632, U$691, U$750, U$809, U$868, U$927, U$986: (no value), output:210
- added U$1046, U$1105, U$1164, U$1223, U$1282, U$1341, U$1400, U$397, U$456, U$515, U$574, U$633, U$692, U$751, U$810, U$869, U$928, U$987: (no value), output:#RST#0
- added U$1047, U$1106, U$1165, U$1224, U$1283, U$1342, U$1401, U$398, U$457, U$516, U$575, U$634, U$693, U$752, U$811, U$870, U$929, U$988: (no value), output:3V3_0
- added U$1049, U$1108, U$1167, U$1226, U$1285, U$1344, U$1403, U$400, U$459, U$518, U$577, U$636, U$695, U$754, U$813, U$872, U$931, U$990: (no value), output:RAW0
- added U$1050, U$1109, U$1168, U$1227, U$1286, U$1345, U$1404, U$401, U$460, U$519, U$578, U$637, U$696, U$755, U$814, U$873, U$932, U$991: (no value), output:R0
- added U$1051, U$1110, U$1169, U$1228, U$1287, U$1346, U$1405, U$402, U$461, U$520, U$579, U$638, U$697, U$756, U$815, U$874, U$933, U$992: (no value), output:#0
- added U$1052, U$1111, U$1170, U$1229, U$1288, U$1347, U$1406, U$403, U$462, U$521, U$580, U$639, U$698, U$757, U$816, U$875, U$934, U$993: (no value), output:PRO_MICRO0
- added U$1053, U$1112, U$1171, U$1230, U$1289, U$1348, U$1407, U$404, U$463, U$522, U$581, U$640, U$699, U$758, U$817, U$876, U$935, U$994: (no value), output:C0
- added U$1054, U$1113, U$1172, U$1231, U$1290, U$1349, U$1408, U$405, U$464, U$523, U$582, U$641, U$700, U$759, U$818, U$877, U$936, U$995: (no value), output:D1
- added U$1055, U$1114, U$1173, U$1232, U$1291, U$1350, U$1409, U$406, U$465, U$524, U$583, U$642, U$701, U$760, U$819, U$878, U$937, U$996: (no value), output:DO0
- added U$1057, U$1116, U$1175, U$1234, U$1293, U$1352, U$1411, U$408, U$467, U$526, U$585, U$644, U$703, U$762, U$821, U$880, U$939, U$998: (no value), output:B0
- added U$1058, U$1117, U$1176, U$1235, U$1294, U$1353, U$1412, U$409, U$468, U$527, U$586, U$645, U$704, U$763, U$822, U$881, U$940, U$999: (no value), output:#SHLD#0
- added U100, U105, U110, U115, U120, U35, U40, U45, U50, U55, U60, U65, U70, U75, U80, U85, U90, U95: APS6404L-3SQR-ZR, RP2350A:APS6404L-3SQR-ZR
- added U101, U106, U111, U116, U31, U36, U41, U46, U51, U56, U61, U66, U71, U76, U81, U86, U91, U96: RT9080-33GJ5, SparkFun-IC-Power:SOT23-5
- added U102, U107, U112, U117, U32, U37, U42, U47, U52, U57, U62, U67, U72, U77, U82, U87, U92, U97: W25QXX128MBIT, SparkFun-IC-Memory:WSON-8-6X5-SKINNY_CENTERPAD
- added U103, U108, U113, U118, U33, U38, U43, U48, U53, U58, U63, U68, U73, U78, U83, U88, U93, U98: WS2812_2020, SparkFun-LED:WS2812-2020
- added U104, U109, U114, U119, U34, U39, U44, U49, U54, U59, U64, U69, U74, U79, U84, U89, U94, U99: RP2350A, RP2350A:RP2350A
- added Y10, Y11, Y12, Y13, Y14, Y15, Y16, Y17, Y18, Y19, Y20, Y21, Y22, Y23, Y24, Y7, Y8, Y9: 12MHz, SparkFun-Clocks:CRYSTAL-SMD-2X2.5MM
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Connections:
- new net !RESET!10: J43.3, J43.3B, R132.1, S21.3, S21.4, U54.26
- new net !RESET!11: J47.3, J47.3B, R145.1, S23.3, S23.4, U59.26
- new net !RESET!12: J51.3, J51.3B, R158.1, S25.3, S25.4, U64.26
- new net !RESET!13: J55.3, J55.3B, R171.1, S27.3, S27.4, U69.26
- new net !RESET!14: J59.3, J59.3B, R184.1, S29.3, S29.4, U74.26
- new net !RESET!15: J63.3, J63.3B, R197.1, S31.3, S31.4, U79.26
- new net !RESET!16: J67.3, J67.3B, R210.1, S33.3, S33.4, U84.26
- new net !RESET!17: J71.3, J71.3B, R223.1, S35.3, S35.4, U89.26
- new net !RESET!18: J75.3, J75.3B, R236.1, S37.3, S37.4, U94.26
- new net !RESET!19: J79.3, J79.3B, R249.1, S39.3, S39.4, U99.26
- new net !RESET!20: J83.3, J83.3B, R262.1, S41.3, S41.4, U104.26
- new net !RESET!21: J87.3, J87.3B, R275.1, S43.3, S43.4, U109.26
- new net !RESET!22: J91.3, J91.3B, R288.1, S45.3, S45.4, U114.26
- new net !RESET!23: J95.3, J95.3B, R301.1, S47.3, S47.4, U119.26
- new net !RESET!6: J27.3, J27.3B, R80.1, S13.3, S13.4, U34.26
- new net !RESET!7: J31.3, J31.3B, R93.1, S15.3, S15.4, U39.26
- new net !RESET!8: J35.3, J35.3B, R106.1, S17.3, S17.4, U44.26
- new net !RESET!9: J39.3, J39.3B, R119.1, S19.3, S19.4, U49.26
- new net 0/TX10: J42.12, J42.12B, U54.2
- new net 0/TX11: J46.12, J46.12B, U59.2
- new net 0/TX12: J50.12, J50.12B, U64.2
- new net 0/TX13: J54.12, J54.12B, U69.2
- new net 0/TX14: J58.12, J58.12B, U74.2
- new net 0/TX15: J62.12, J62.12B, U79.2
- new net 0/TX16: J66.12, J66.12B, U84.2
- new net 0/TX17: J70.12, J70.12B, U89.2
- new net 0/TX18: J74.12, J74.12B, U94.2
- new net 0/TX19: J78.12, J78.12B, U99.2
- new net 0/TX20: J82.12, J82.12B, U104.2
- new net 0/TX21: J86.12, J86.12B, U109.2
- new net 0/TX22: J90.12, J90.12B, U114.2
- new net 0/TX23: J94.12, J94.12B, U119.2
- new net 0/TX6: J26.12, J26.12B, U34.2
- new net 0/TX7: J30.12, J30.12B, U39.2
- new net 0/TX8: J34.12, J34.12B, U44.2
- new net 0/TX9: J38.12, J38.12B, U49.2
- new net 1.1V10: C211.1, C212.1, C213.1, C218.1, L11.1, U54.23, U54.39, U54.50, U54.6
- new net 1.1V11: C231.1, C232.1, C233.1, C238.1, L12.1, U59.23, U59.39, U59.50, U59.6
- new net 1.1V12: C251.1, C252.1, C253.1, C258.1, L13.1, U64.23, U64.39, U64.50, U64.6
- new net 1.1V13: C271.1, C272.1, C273.1, C278.1, L14.1, U69.23, U69.39, U69.50, U69.6
- new net 1.1V14: C291.1, C292.1, C293.1, C298.1, L15.1, U74.23, U74.39, U74.50, U74.6
- new net 1.1V15: C311.1, C312.1, C313.1, C318.1, L16.1, U79.23, U79.39, U79.50, U79.6
- new net 1.1V16: C331.1, C332.1, C333.1, C338.1, L17.1, U84.23, U84.39, U84.50, U84.6
- new net 1.1V17: C351.1, C352.1, C353.1, C358.1, L18.1, U89.23, U89.39, U89.50, U89.6
- new net 1.1V18: C371.1, C372.1, C373.1, C378.1, L19.1, U94.23, U94.39, U94.50, U94.6
- new net 1.1V19: C391.1, C392.1, C393.1, C398.1, L20.1, U99.23, U99.39, U99.50, U99.6
- new net 1.1V20: C411.1, C412.1, C413.1, C418.1, L21.1, U104.23, U104.39, U104.50, U104.6
- new net 1.1V21: C431.1, C432.1, C433.1, C438.1, L22.1, U109.23, U109.39, U109.50, U109.6
- new net 1.1V22: C451.1, C452.1, C453.1, C458.1, L23.1, U114.23, U114.39, U114.50, U114.6
- new net 1.1V23: C471.1, C472.1, C473.1, C478.1, L24.1, U119.23, U119.39, U119.50, U119.6
- new net 1.1V6: C131.1, C132.1, C133.1, C138.1, L7.1, U34.23, U34.39, U34.50, U34.6
- new net 1.1V7: C151.1, C152.1, C153.1, C158.1, L8.1, U39.23, U39.39, U39.50, U39.6
- new net 1.1V8: C171.1, C172.1, C173.1, C178.1, L9.1, U44.23, U44.39, U44.50, U44.6
- new net 1.1V9: C191.1, C192.1, C193.1, C198.1, L10.1, U49.23, U49.39, U49.50, U49.6
- new net 1/RX10: J42.11, J42.11B, U54.3
- new net 1/RX11: J46.11, J46.11B, U59.3
- new net 1/RX12: J50.11, J50.11B, U64.3
- new net 1/RX13: J54.11, J54.11B, U69.3
- new net 1/RX14: J58.11, J58.11B, U74.3
- new net 1/RX15: J62.11, J62.11B, U79.3
- new net 1/RX16: J66.11, J66.11B, U84.3
- new net 1/RX17: J70.11, J70.11B, U89.3
- new net 1/RX18: J74.11, J74.11B, U94.3
- new net 1/RX19: J78.11, J78.11B, U99.3
- new net 1/RX20: J82.11, J82.11B, U104.3
- new net 1/RX21: J86.11, J86.11B, U109.3
- new net 1/RX22: J90.11, J90.11B, U114.3
- new net 1/RX23: J94.11, J94.11B, U119.3
- new net 1/RX6: J26.11, J26.11B, U34.3
- new net 1/RX7: J30.11, J30.11B, U39.3
- new net 1/RX8: J34.11, J34.11B, U44.3
- new net 1/RX9: J38.11, J38.11B, U49.3
- new net 100: J66.3, J66.3B, U84.10
- new net 101: J66.8, J66.8B, U84.4
- new net 102: J66.7, J66.7B, U84.5
- new net 103: J70.5, J70.5B, U89.8
- new net 104: J70.6, J70.6B, U89.7
- new net 105: J70.4, J70.4B, U89.9
- new net 106: J70.3, J70.3B, U89.10
- new net 107: J70.8, J70.8B, U89.4
- new net 108: J70.7, J70.7B, U89.5
- new net 109: J74.5, J74.5B, U94.8
- new net 110: J74.6, J74.6B, U94.7
- new net 111: J74.4, J74.4B, U94.9
- new net 112: J74.3, J74.3B, U94.10
- new net 113: J74.8, J74.8B, U94.4
- new net 114: J74.7, J74.7B, U94.5
- new net 115: J78.5, J78.5B, U99.8
- new net 116: J78.6, J78.6B, U99.7
- new net 117: J78.4, J78.4B, U99.9
- new net 118: J78.3, J78.3B, U99.10
- new net 119: J78.8, J78.8B, U99.4
- new net 120: J78.7, J78.7B, U99.5
- new net 121: J82.5, J82.5B, U104.8
- new net 122: J82.6, J82.6B, U104.7
- new net 123: J82.4, J82.4B, U104.9
- new net 124: J82.3, J82.3B, U104.10
- new net 125: J82.8, J82.8B, U104.4
- new net 126: J82.7, J82.7B, U104.5
- new net 127: J86.5, J86.5B, U109.8
- new net 128: J86.6, J86.6B, U109.7
- new net 129: J86.4, J86.4B, U109.9
- new net 130: J86.3, J86.3B, U109.10
- new net 131: J86.8, J86.8B, U109.4
- new net 132: J86.7, J86.7B, U109.5
- new net 133: J90.5, J90.5B, U114.8
- new net 134: J90.6, J90.6B, U114.7
- new net 135: J90.4, J90.4B, U114.9
- new net 136: J90.3, J90.3B, U114.10
- new net 137: J90.8, J90.8B, U114.4
- new net 138: J90.7, J90.7B, U114.5
- new net 139: J94.5, J94.5B, U119.8
- new net 140: J94.6, J94.6B, U119.7
- new net 141: J94.4, J94.4B, U119.9
- new net 142: J94.3, J94.3B, U119.10
- new net 143: J94.8, J94.8B, U119.4
- new net 144: J94.7, J94.7B, U119.5
- new net 16/SDA10: J41.3, R135.1, U54.27
- new net 16/SDA11: J45.3, R148.1, U59.27
- new net 16/SDA12: J49.3, R161.1, U64.27
- new net 16/SDA13: J53.3, R174.1, U69.27
- new net 16/SDA14: J57.3, R187.1, U74.27
- new net 16/SDA15: J61.3, R200.1, U79.27
- new net 16/SDA16: J65.3, R213.1, U84.27
- new net 16/SDA17: J69.3, R226.1, U89.27
- new net 16/SDA18: J73.3, R239.1, U94.27
- new net 16/SDA19: J77.3, R252.1, U99.27
- new net 16/SDA20: J81.3, R265.1, U104.27
- new net 16/SDA21: J85.3, R278.1, U109.27
- new net 16/SDA22: J89.3, R291.1, U114.27
- new net 16/SDA23: J93.3, R304.1, U119.27
- new net 16/SDA6: J25.3, R83.1, U34.27
- new net 16/SDA7: J29.3, R96.1, U39.27
- new net 16/SDA8: J33.3, R109.1, U44.27
- new net 16/SDA9: J37.3, R122.1, U49.27
- new net 17/SCL10: J41.4, R136.1, U54.28
- new net 17/SCL11: J45.4, R149.1, U59.28
- new net 17/SCL12: J49.4, R162.1, U64.28
- new net 17/SCL13: J53.4, R175.1, U69.28
- new net 17/SCL14: J57.4, R188.1, U74.28
- new net 17/SCL15: J61.4, R201.1, U79.28
- new net 17/SCL16: J65.4, R214.1, U84.28
- new net 17/SCL17: J69.4, R227.1, U89.28
- new net 17/SCL18: J73.4, R240.1, U94.28
- new net 17/SCL19: J77.4, R253.1, U99.28
- new net 17/SCL20: J81.4, R266.1, U104.28
- new net 17/SCL21: J85.4, R279.1, U109.28
- new net 17/SCL22: J89.4, R292.1, U114.28
- new net 17/SCL23: J93.4, R305.1, U119.28
- new net 17/SCL6: J25.4, R84.1, U34.28
- new net 17/SCL7: J29.4, R97.1, U39.28
- new net 17/SCL8: J33.4, R110.1, U44.28
- new net 17/SCL9: J37.4, R123.1, U49.28
- new net 20/SPI_POCI10: J43.10, J43.10B, U54.32
- new net 20/SPI_POCI11: J47.10, J47.10B, U59.32
- new net 20/SPI_POCI12: J51.10, J51.10B, U64.32
- new net 20/SPI_POCI13: J55.10, J55.10B, U69.32
- new net 20/SPI_POCI14: J59.10, J59.10B, U74.32
- new net 20/SPI_POCI15: J63.10, J63.10B, U79.32
- new net 20/SPI_POCI16: J67.10, J67.10B, U84.32
- new net 20/SPI_POCI17: J71.10, J71.10B, U89.32
- new net 20/SPI_POCI18: J75.10, J75.10B, U94.32
- new net 20/SPI_POCI19: J79.10, J79.10B, U99.32
- new net 20/SPI_POCI20: J83.10, J83.10B, U104.32
- new net 20/SPI_POCI21: J87.10, J87.10B, U109.32
- new net 20/SPI_POCI22: J91.10, J91.10B, U114.32
- new net 20/SPI_POCI23: J95.10, J95.10B, U119.32
- new net 20/SPI_POCI6: J27.10, J27.10B, U34.32
- new net 20/SPI_POCI7: J31.10, J31.10B, U39.32
- new net 20/SPI_POCI8: J35.10, J35.10B, U44.32
- new net 20/SPI_POCI9: J39.10, J39.10B, U49.32
- new net 21/SPI_!CS!10: J43.12, J43.12B, U54.33
- new net 21/SPI_!CS!11: J47.12, J47.12B, U59.33
- new net 21/SPI_!CS!12: J51.12, J51.12B, U64.33
- new net 21/SPI_!CS!13: J55.12, J55.12B, U69.33
- new net 21/SPI_!CS!14: J59.12, J59.12B, U74.33
- new net 21/SPI_!CS!15: J63.12, J63.12B, U79.33
- new net 21/SPI_!CS!16: J67.12, J67.12B, U84.33
- new net 21/SPI_!CS!17: J71.12, J71.12B, U89.33
- new net 21/SPI_!CS!18: J75.12, J75.12B, U94.33
- new net 21/SPI_!CS!19: J79.12, J79.12B, U99.33
- new net 21/SPI_!CS!20: J83.12, J83.12B, U104.33
- new net 21/SPI_!CS!21: J87.12, J87.12B, U109.33
- new net 21/SPI_!CS!22: J91.12, J91.12B, U114.33
- new net 21/SPI_!CS!23: J95.12, J95.12B, U119.33
- new net 21/SPI_!CS!6: J27.12, J27.12B, U34.33
- new net 21/SPI_!CS!7: J31.12, J31.12B, U39.33
- new net 21/SPI_!CS!8: J35.12, J35.12B, U44.33
- new net 21/SPI_!CS!9: J39.12, J39.12B, U49.33
- new net 22/SPI_SCK10: J43.9, J43.9B, U54.34
- new net 22/SPI_SCK11: J47.9, J47.9B, U59.34
- new net 22/SPI_SCK12: J51.9, J51.9B, U64.34
- new net 22/SPI_SCK13: J55.9, J55.9B, U69.34
- new net 22/SPI_SCK14: J59.9, J59.9B, U74.34
- new net 22/SPI_SCK15: J63.9, J63.9B, U79.34
- new net 22/SPI_SCK16: J67.9, J67.9B, U84.34
- new net 22/SPI_SCK17: J71.9, J71.9B, U89.34
- new net 22/SPI_SCK18: J75.9, J75.9B, U94.34
- new net 22/SPI_SCK19: J79.9, J79.9B, U99.34
- new net 22/SPI_SCK20: J83.9, J83.9B, U104.34
- new net 22/SPI_SCK21: J87.9, J87.9B, U109.34
- new net 22/SPI_SCK22: J91.9, J91.9B, U114.34
- new net 22/SPI_SCK23: J95.9, J95.9B, U119.34
- new net 22/SPI_SCK6: J27.9, J27.9B, U34.34
- new net 22/SPI_SCK7: J31.9, J31.9B, U39.34
- new net 22/SPI_SCK8: J35.9, J35.9B, U44.34
- new net 22/SPI_SCK9: J39.9, J39.9B, U49.34
- new net 23/SPI_PICO10: J43.11, J43.11B, U54.35
- new net 23/SPI_PICO11: J47.11, J47.11B, U59.35
- new net 23/SPI_PICO12: J51.11, J51.11B, U64.35
- new net 23/SPI_PICO13: J55.11, J55.11B, U69.35
- new net 23/SPI_PICO14: J59.11, J59.11B, U74.35
- new net 23/SPI_PICO15: J63.11, J63.11B, U79.35
- new net 23/SPI_PICO16: J67.11, J67.11B, U84.35
- new net 23/SPI_PICO17: J71.11, J71.11B, U89.35
- new net 23/SPI_PICO18: J75.11, J75.11B, U94.35
- new net 23/SPI_PICO19: J79.11, J79.11B, U99.35
- new net 23/SPI_PICO20: J83.11, J83.11B, U104.35
- new net 23/SPI_PICO21: J87.11, J87.11B, U109.35
- new net 23/SPI_PICO22: J91.11, J91.11B, U114.35
- new net 23/SPI_PICO23: J95.11, J95.11B, U119.35
- new net 23/SPI_PICO6: J27.11, J27.11B, U34.35
- new net 23/SPI_PICO7: J31.11, J31.11B, U39.35
- new net 23/SPI_PICO8: J35.11, J35.11B, U44.35
- new net 23/SPI_PICO9: J39.11, J39.11B, U49.35
- new net 25/WS2812-DI10: U53.DI, U54.37
- new net 25/WS2812-DI11: U58.DI, U59.37
- new net 25/WS2812-DI12: U63.DI, U64.37
- new net 25/WS2812-DI13: U68.DI, U69.37
- new net 25/WS2812-DI14: U73.DI, U74.37
- new net 25/WS2812-DI15: U78.DI, U79.37
- new net 25/WS2812-DI16: U83.DI, U84.37
- new net 25/WS2812-DI17: U88.DI, U89.37
- new net 25/WS2812-DI18: U93.DI, U94.37
- new net 25/WS2812-DI19: U98.DI, U99.37
- new net 25/WS2812-DI20: U103.DI, U104.37
- new net 25/WS2812-DI21: U108.DI, U109.37
- new net 25/WS2812-DI22: U113.DI, U114.37
- new net 25/WS2812-DI23: U118.DI, U119.37
- new net 25/WS2812-DI6: U33.DI, U34.37
- new net 25/WS2812-DI7: U38.DI, U39.37
- new net 25/WS2812-DI8: U43.DI, U44.37
- new net 25/WS2812-DI9: U48.DI, U49.37
- new net 3.3V10: C202.2, C205.1, C206.1, C207.1, C208.1, C209.1, C210.1, C214.1, C216.1, C217.1, C219.1, C220.1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
- new net 3.3V11: C222.2, C225.1, C226.1, C227.1, C228.1, C229.1, C230.1, C234.1, C236.1, C237.1, C239.1, C240.1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
- new net 3.3V12: C242.2, C245.1, C246.1, C247.1, C248.1, C249.1, C250.1, C254.1, C256.1, C257.1, C259.1, C260.1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
- new net 3.3V13: C262.2, C265.1, C266.1, C267.1, C268.1, C269.1, C270.1, C274.1, C276.1, C277.1, C279.1, C280.1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
- new net 3.3V14: C282.2, C285.1, C286.1, C287.1, C288.1, C289.1, C290.1, C294.1, C296.1, C297.1, C299.1, C300.1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
- new net 3.3V15: C302.2, C305.1, C306.1, C307.1, C308.1, C309.1, C310.1, C314.1, C316.1, C317.1, C319.1, C320.1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
- new net 3.3V16: C322.2, C325.1, C326.1, C327.1, C328.1, C329.1, C330.1, C334.1, C336.1, C337.1, C339.1, C340.1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
- new net 3.3V17: C342.2, C345.1, C346.1, C347.1, C348.1, C349.1, C350.1, C354.1, C356.1, C357.1, C359.1, C360.1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
- new net 3.3V18: C362.2, C365.1, C366.1, C367.1, C368.1, C369.1, C370.1, C374.1, C376.1, C377.1, C379.1, C380.1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
- new net 3.3V19: C382.2, C385.1, C386.1, C387.1, C388.1, C389.1, C390.1, C394.1, C396.1, C397.1, C399.1, C400.1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
- new net 3.3V20: C402.2, C405.1, C406.1, C407.1, C408.1, C409.1, C410.1, C414.1, C416.1, C417.1, C419.1, C420.1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
- new net 3.3V21: C422.2, C425.1, C426.1, C427.1, C428.1, C429.1, C430.1, C434.1, C436.1, C437.1, C439.1, C440.1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
- new net 3.3V22: C442.2, C445.1, C446.1, C447.1, C448.1, C449.1, C450.1, C454.1, C456.1, C457.1, C459.1, C460.1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
- new net 3.3V23: C462.2, C465.1, C466.1, C467.1, C468.1, C469.1, C470.1, C474.1, C476.1, C477.1, C479.1, C480.1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
- new net 3.3V6: C122.2, C125.1, C126.1, C127.1, C128.1, C129.1, C130.1, C134.1, C136.1, C137.1, C139.1, C140.1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
- new net 3.3V7: C142.2, C145.1, C146.1, C147.1, C148.1, C149.1, C150.1, C154.1, C156.1, C157.1, C159.1, C160.1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
- new net 3.3V8: C162.2, C165.1, C166.1, C167.1, C168.1, C169.1, C170.1, C174.1, C176.1, C177.1, C179.1, C180.1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
- new net 3.3V9: C182.2, C185.1, C186.1, C187.1, C188.1, C189.1, C190.1, C194.1, C196.1, C197.1, C199.1, C200.1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
- new net 37: J26.5, J26.5B, U34.8
- new net 38: J26.6, J26.6B, U34.7
- new net 39: J26.4, J26.4B, U34.9
- new net 40: J26.3, J26.3B, U34.10
- new net 41: J26.8, J26.8B, U34.4
- new net 42: J26.7, J26.7B, U34.5
- new net 43: J30.5, J30.5B, U39.8
- new net 44: J30.6, J30.6B, U39.7
- new net 45: J30.4, J30.4B, U39.9
- new net 46: J30.3, J30.3B, U39.10
- new net 47: J30.8, J30.8B, U39.4
- new net 48: J30.7, J30.7B, U39.5
- new net 49: J34.5, J34.5B, U44.8
- new net 50: J34.6, J34.6B, U44.7
- new net 51: J34.4, J34.4B, U44.9
- new net 52: J34.3, J34.3B, U44.10
- new net 53: J34.8, J34.8B, U44.4
- new net 54: J34.7, J34.7B, U44.5
- new net 55: J38.5, J38.5B, U49.8
- new net 56: J38.6, J38.6B, U49.7
- new net 57: J38.4, J38.4B, U49.9
- new net 58: J38.3, J38.3B, U49.10
- new net 59: J38.8, J38.8B, U49.4
- new net 60: J38.7, J38.7B, U49.5
- new net 61: J42.5, J42.5B, U54.8
- new net 62: J42.6, J42.6B, U54.7
- new net 63: J42.4, J42.4B, U54.9
- new net 64: J42.3, J42.3B, U54.10
- new net 65: J42.8, J42.8B, U54.4
- new net 66: J42.7, J42.7B, U54.5
- new net 67: J46.5, J46.5B, U59.8
- new net 68: J46.6, J46.6B, U59.7
- new net 69: J46.4, J46.4B, U59.9
- new net 70: J46.3, J46.3B, U59.10
- new net 71: J46.8, J46.8B, U59.4
- new net 72: J46.7, J46.7B, U59.5
- new net 73: J50.5, J50.5B, U64.8
- new net 74: J50.6, J50.6B, U64.7
- new net 75: J50.4, J50.4B, U64.9
- new net 76: J50.3, J50.3B, U64.10
- new net 77: J50.8, J50.8B, U64.4
- new net 78: J50.7, J50.7B, U64.5
- new net 79: J54.5, J54.5B, U69.8
- new net 8/TX10: J38.2, J38.2B, U49.12
- new net 8/TX11: J42.2, J42.2B, U54.12
- new net 8/TX12: J46.2, J46.2B, U59.12
- new net 8/TX13: J50.2, J50.2B, U64.12
- new net 8/TX14: J54.2, J54.2B, U69.12
- new net 8/TX15: J58.2, J58.2B, U74.12
- new net 8/TX16: J62.2, J62.2B, U79.12
- new net 8/TX17: J66.2, J66.2B, U84.12
- new net 8/TX18: J70.2, J70.2B, U89.12
- new net 8/TX19: J74.2, J74.2B, U94.12
- new net 8/TX20: J78.2, J78.2B, U99.12
- new net 8/TX21: J82.2, J82.2B, U104.12
- new net 8/TX22: J86.2, J86.2B, U109.12
- new net 8/TX23: J90.2, J90.2B, U114.12
- new net 8/TX24: J94.2, J94.2B, U119.12
- new net 8/TX7: J26.2, J26.2B, U34.12
- new net 8/TX8: J30.2, J30.2B, U39.12
- new net 8/TX9: J34.2, J34.2B, U44.12
- new net 80: J54.6, J54.6B, U69.7
- new net 81: J54.4, J54.4B, U69.9
- new net 82: J54.3, J54.3B, U69.10
- new net 83: J54.8, J54.8B, U69.4
- new net 84: J54.7, J54.7B, U69.5
- new net 85: J58.5, J58.5B, U74.8
- new net 86: J58.6, J58.6B, U74.7
- new net 87: J58.4, J58.4B, U74.9
- new net 88: J58.3, J58.3B, U74.10
- new net 89: J58.8, J58.8B, U74.4
- new net 9/RX10: J38.1, J38.1B, U49.13
- new net 9/RX11: J42.1, J42.1B, U54.13
- new net 9/RX12: J46.1, J46.1B, U59.13
- new net 9/RX13: J50.1, J50.1B, U64.13
- new net 9/RX14: J54.1, J54.1B, U69.13
- new net 9/RX15: J58.1, J58.1B, U74.13
- new net 9/RX16: J62.1, J62.1B, U79.13
- new net 9/RX17: J66.1, J66.1B, U84.13
- new net 9/RX18: J70.1, J70.1B, U89.13
- new net 9/RX19: J74.1, J74.1B, U94.13
- new net 9/RX20: J78.1, J78.1B, U99.13
- new net 9/RX21: J82.1, J82.1B, U104.13
- new net 9/RX22: J86.1, J86.1B, U109.13
- new net 9/RX23: J90.1, J90.1B, U114.13
- new net 9/RX24: J94.1, J94.1B, U119.13
- new net 9/RX7: J26.1, J26.1B, U34.13
- new net 9/RX8: J30.1, J30.1B, U39.13
- new net 9/RX9: J34.1, J34.1B, U44.13
- new net 90: J58.7, J58.7B, U74.5
- new net 91: J62.5, J62.5B, U79.8
- new net 92: J62.6, J62.6B, U79.7
- new net 93: J62.4, J62.4B, U79.9
- new net 94: J62.3, J62.3B, U79.10
- new net 95: J62.8, J62.8B, U79.4
- new net 96: J62.7, J62.7B, U79.5
- new net 97: J66.5, J66.5B, U84.8
- new net 98: J66.6, J66.6B, U84.7
- new net 99: J66.4, J66.4B, U84.9
- new net A24: J27.5, J27.5B, U34.43
- new net A25: J27.6, J27.6B, U34.42
- new net A26: J27.7, J27.7B, U34.41
- new net A27: J27.8, J27.8B, U34.40
- new net A28: J31.5, J31.5B, U39.43
- new net A29: J31.6, J31.6B, U39.42
- new net A30: J31.7, J31.7B, U39.41
- new net A31: J31.8, J31.8B, U39.40
- new net A32: J35.5, J35.5B, U44.43
- new net A33: J35.6, J35.6B, U44.42
- new net A34: J35.7, J35.7B, U44.41
- new net A35: J35.8, J35.8B, U44.40
- new net A36: J39.5, J39.5B, U49.43
- new net A37: J39.6, J39.6B, U49.42
- new net A38: J39.7, J39.7B, U49.41
- new net A39: J39.8, J39.8B, U49.40
- new net A40: J43.5, J43.5B, U54.43
- new net A41: J43.6, J43.6B, U54.42
- new net A42: J43.7, J43.7B, U54.41
- new net A43: J43.8, J43.8B, U54.40
- new net A44: J47.5, J47.5B, U59.43
- new net A45: J47.6, J47.6B, U59.42
- new net A46: J47.7, J47.7B, U59.41
- new net A47: J47.8, J47.8B, U59.40
- new net A48: J51.5, J51.5B, U64.43
- new net A49: J51.6, J51.6B, U64.42
- new net A50: J51.7, J51.7B, U64.41
- new net A51: J51.8, J51.8B, U64.40
- new net A52: J55.5, J55.5B, U69.43
- new net A53: J55.6, J55.6B, U69.42
- new net A54: J55.7, J55.7B, U69.41
- new net A55: J55.8, J55.8B, U69.40
- new net A56: J59.5, J59.5B, U74.43
- new net A57: J59.6, J59.6B, U74.42
- new net A58: J59.7, J59.7B, U74.41
- new net A59: J59.8, J59.8B, U74.40
- new net A60: J63.5, J63.5B, U79.43
- new net A61: J63.6, J63.6B, U79.42
- new net A62: J63.7, J63.7B, U79.41
- new net A63: J63.8, J63.8B, U79.40
- new net A64: J67.5, J67.5B, U84.43
- new net A65: J67.6, J67.6B, U84.42
- new net A66: J67.7, J67.7B, U84.41
- new net A67: J67.8, J67.8B, U84.40
- new net A68: J71.5, J71.5B, U89.43
- new net A69: J71.6, J71.6B, U89.42
- new net A70: J71.7, J71.7B, U89.41
- new net A71: J71.8, J71.8B, U89.40
- new net A72: J75.5, J75.5B, U94.43
- new net A73: J75.6, J75.6B, U94.42
- new net A74: J75.7, J75.7B, U94.41
- new net A75: J75.8, J75.8B, U94.40
- new net A76: J79.5, J79.5B, U99.43
- new net A77: J79.6, J79.6B, U99.42
- new net A78: J79.7, J79.7B, U99.41
- new net A79: J79.8, J79.8B, U99.40
- new net A80: J83.5, J83.5B, U104.43
- new net A81: J83.6, J83.6B, U104.42
- new net A82: J83.7, J83.7B, U104.41
- new net A83: J83.8, J83.8B, U104.40
- new net A84: J87.5, J87.5B, U109.43
- new net A85: J87.6, J87.6B, U109.42
- new net A86: J87.7, J87.7B, U109.41
- new net A87: J87.8, J87.8B, U109.40
- new net A88: J91.5, J91.5B, U114.43
- new net A89: J91.6, J91.6B, U114.42
- new net A90: J91.7, J91.7B, U114.41
- new net A91: J91.8, J91.8B, U114.40
- new net A92: J95.5, J95.5B, U119.43
- new net A93: J95.6, J95.6B, U119.42
- new net A94: J95.7, J95.7B, U119.41
- new net A95: J95.8, J95.8B, U119.40
- new net BOOT10: R141.2, S22.3, S22.4, TP44.1
- new net BOOT11: R154.2, S24.3, S24.4, TP48.1
- new net BOOT12: R167.2, S26.3, S26.4, TP52.1
- new net BOOT13: R180.2, S28.3, S28.4, TP56.1
- new net BOOT14: R193.2, S30.3, S30.4, TP60.1
- new net BOOT15: R206.2, S32.3, S32.4, TP64.1
- new net BOOT16: R219.2, S34.3, S34.4, TP68.1
- new net BOOT17: R232.2, S36.3, S36.4, TP72.1
- new net BOOT18: R245.2, S38.3, S38.4, TP76.1
- new net BOOT19: R258.2, S40.3, S40.4, TP80.1
- new net BOOT20: R271.2, S42.3, S42.4, TP84.1
- new net BOOT21: R284.2, S44.3, S44.4, TP88.1
- new net BOOT22: R297.2, S46.3, S46.4, TP92.1
- new net BOOT23: R310.2, S48.3, S48.4, TP96.1
- new net BOOT6: R89.2, S14.3, S14.4, TP28.1
- new net BOOT7: R102.2, S16.3, S16.4, TP32.1
- new net BOOT8: R115.2, S18.3, S18.4, TP36.1
- new net BOOT9: R128.2, S20.3, S20.4, TP40.1
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Routing:
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- added copper zone on layer 1, net 1.1V10
- added copper zone on layer 1, net 1.1V11
- added copper zone on layer 1, net 1.1V12
- added copper zone on layer 1, net 1.1V13
- added copper zone on layer 1, net 1.1V14
- added copper zone on layer 1, net 1.1V15
- added copper zone on layer 1, net 1.1V16
- added copper zone on layer 1, net 1.1V17
- added copper zone on layer 1, net 1.1V18
- added copper zone on layer 1, net 1.1V19
- added copper zone on layer 1, net 1.1V20
- added copper zone on layer 1, net 1.1V21
- added copper zone on layer 1, net 1.1V22
- added copper zone on layer 1, net 1.1V23
- added copper zone on layer 1, net 1.1V6
- added copper zone on layer 1, net 1.1V7
- added copper zone on layer 1, net 1.1V8
- added copper zone on layer 1, net 1.1V9
- added copper zone on layer 1, net 3.3V10
- added copper zone on layer 15, net 3.3V10
- added copper zone on layer 1, net 3.3V11
- added copper zone on layer 15, net 3.3V11
- added copper zone on layer 1, net 3.3V12
- added copper zone on layer 15, net 3.3V12
- added copper zone on layer 1, net 3.3V13
- added copper zone on layer 15, net 3.3V13
- added copper zone on layer 1, net 3.3V14
- added copper zone on layer 15, net 3.3V14
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Other:
- board size 92.7 x 87.1 mm -> 200.7 x 125.5 mm
- board text added: "v10"
- board text removed: "v-score"
- board text removed: "v02"
